Commit message: Changed from rotational to fixed the joint between the rotational robot holder and the robot

File: src/gazebo_resources/models/rotational_robot_holder/urdf/rotational_robot_holder.xacro (robot description, xacro)
@@ -52,10 +52,8 @@
     <dynamics damping="0.7"/>
   </joint>
-  <joint name="rotational_robot_holder_to_rotot" type="continuous">
+  <joint name="rotational_robot_holder_to_rotot" type="fixed">
     <parent link="rotational_robot_holder_holder"/>
     <child link="body"/>
     <origin xyz="${rotational_robot_holder_holder_length} 0 0" rpy="0 0 0"/>
-    <axis xyz="1 0 0"/>
-    <dynamics damping="0.7"/>
   </joint>
 </robot>

Commit message: Added an extra dof to allow movemnt in z axis

File: src/gazebo_resources/models/rotational_robot_holder/urdf/rotational_robot_holder.xacro (robot description, xacro)
@@ -18,4 +18,23 @@
       <mass value="10"/>
       <inertia ixx="0.4" ixy="0.0" ixz="0.0" iyy="0.4" iyz="0.0" izz="0.2"/>
+    </inertial>
+  </link>
+  <link name="rotational_robot_holder_virtual">
+    <collision>
+      <origin xyz="0 0 0" rpy="0 0 0"/>
+      <geometry>
+        <sphere radius="0.01"/>
+      </geometry>
+    </collision>
+    <visual>
+      <origin xyz="0 0 0" rpy="0 0 0"/>
+      <geometry>
+         <sphere radius="0.01"/>
+      </geometry>
+      <material name="orange"/>
+    </visual>
+    <inertial>
+      <mass value="0.01"/>
+      <inertia ixx="0.1" ixy="0.0" ixz="0.0" iyy="0.1" iyz="0.0" izz="0.1"/>
     </inertial>
   </link>
@@ -45,6 +64,13 @@
     <origin xyz="0 0 ${rotational_robot_holder_base_length/2}" rpy="0 0 0"/>
   </joint>
+  <joint name="rotational_robot_holder_virtual_to_holder" type="continuous">
+    <parent link="rotational_robot_holder_base"/>
+    <child link="rotational_robot_holder_virtual"/>
+    <origin xyz="0 0 0" rpy="0 0 0"/>
+    <axis xyz="0 1 0"/>
+    <dynamics damping="0.7"/>
+  </joint>
   <joint name="rotational_robot_holder_joint" type="continuous">
-    <parent link="rotational_robot_holder_base"/>
+    <parent link="rotational_robot_holder_virtual"/>
     <child link="rotational_robot_holder_holder"/>
     <origin xyz="0 0 ${rotational_robot_holder_base_length/2}" rpy="0 0 0"/>
@@ -56,4 +82,6 @@
     <child link="body"/>
     <origin xyz="${rotational_robot_holder_holder_length} 0 0" rpy="0 0 0"/>
+    <axis xyz="0 0 1"/>
+    <limit effort="30" velocity="1.0" lower="0" upper="1" />
   </joint>
 </robot>

Commit message: Attach the holder to the side of the robot, not the middle

File: src/gazebo_resources/models/rotational_robot_holder/urdf/rotational_robot_holder.xacro (robot description, xacro)
@@ -81,5 +81,5 @@
     <parent link="rotational_robot_holder_holder"/>
     <child link="body"/>
-    <origin xyz="${rotational_robot_holder_holder_length} 0 0" rpy="0 0 0"/>
+    <origin xyz="${rotational_robot_holder_holder_length+bodyWidth/2} 0 0" rpy="0 0 0"/>
     <axis xyz="0 0 1"/>
     <limit effort="30" velocity="1.0" lower="0" upper="1" />
