Commit message: Works in rviz but not in gazebo

File: src/dacbot_description/urdf/dacbot.urdf (robot description, URDF)
Before this commit: robot dacbot, 8 links, 8 joints
Links:
- removed link world
- added link dacbot_origin
Joints:
- removed joint world_left_foot
- removed joint world_right_foot
- added joint dacbot: type fixed, parent dacbot_origin, child body, origin xyz=0 0 0.525 rpy=0 0 0
- joint left_ankle: axis 1 0 0 -> 0 0 1; child left_lower_leg -> left_foot; origin xyz=-0.015 0 0.004 rpy=0 0 0 -> xyz=0.125 0 0 rpy=0 0 0; parent left_foot -> left_lower_leg
- joint left_hip: axis 1 0 0 -> 0 0 1; child body -> left_upper_leg; origin xyz=-0.015 0 0 rpy=0 0 0 -> xyz=-0.015 0 0 rpy=0 1.57079632679 0; parent left_upper_leg -> body
- joint left_knee: axis 1 0 0 -> 0 0 1; child left_upper_leg -> left_lower_leg; origin xyz=-0.015 0 0 rpy=0 0 0 -> xyz=0.142 0 0 rpy=0 0 0; parent left_lower_leg -> left_upper_leg; type fixed -> continuous
- joint right_ankle: axis 1 0 0 -> 0 0 1; child right_lower_leg -> right_foot; origin xyz=-0.015 0 0.004 rpy=0 0 0 -> xyz=0.125 0 0 rpy=0 0 0; parent right_foot -> right_lower_leg
- joint right_hip: axis 1 0 0 -> 0 0 1; child body -> right_upper_leg; origin xyz=-0.015 0 0 rpy=0 0 0 -> xyz=0.015 0 0 rpy=0 1.57079632679 0; parent right_upper_leg -> body
- joint right_knee: axis 1 0 0 -> 0 0 1; child right_upper_leg -> right_lower_leg; origin xyz=-0.015 0 0 rpy=0 0 0 -> xyz=0.142 0 0 rpy=0 0 0; parent right_lower_leg -> right_upper_leg; type fixed -> continuous

File: src/dacbot_description/urdf/dacbot.xacro (robot description, xacro)
@@ -50,10 +50,10 @@
 	 -->
 	 <!-- Box Macro!
-	<xacro:create_box name="" origin_x="" origin_y="" origin_z="" width="" length="" height="" mass="" />
+	<xacro:create_box name="" origin_x="" origin_y="" origin_z="" r="" p="" y="" width="" length="" height="" mass="" />
 	 -->
-	<xacro:macro name="create_box" params="name origin_x origin_y origin_z width length height mass">
+	<xacro:macro name="create_box" params="name origin_x origin_y origin_z r p y width length height mass">
 		<link name="${name}">
 			<collision>
-				<origin xyz="${origin_x} ${origin_y} ${origin_z}" rpy="0 0 0"/>
+				<origin xyz="${origin_x} ${origin_y} ${origin_z}" rpy="${r} ${p} ${y}"/>
 				<geometry>
 					<box size="${width*scale} ${length*scale} ${height*scale}" />
@@ -61,5 +61,5 @@
 			</collision>
 			<visual>
-				<origin xyz="${origin_x} ${origin_y} ${origin_z}" rpy="0 0 0"/>
+				<origin xyz="${origin_x} ${origin_y} ${origin_z}" rpy="${r} ${p} ${y}"/>
 				<geometry>
 					<box size="${width*scale} ${length*scale} ${height*scale}" />
@@ -68,5 +68,5 @@
 			</visual>
 			<inertial>
-				<origin xyz="${origin_x} ${origin_y} ${origin_z}" rpy="0 0 0"/>
+				<origin xyz="${origin_x} ${origin_y} ${origin_z}" rpy="${r} ${p} ${y}"/>
 				<mass value="${mass}"/>
 				<inertia
@@ -78,79 +78,142 @@
 	</xacro:macro>
 	<!--
+		World
+	-->
+	<!-- <link name="dacbot_global"/> -->
+	<!--
 		Left Leg
 	-->
 	<!-- Left Foot -->
-	<xacro:create_box name="left_foot" origin_x="${-legDistFromCenter}" origin_y="${footLength*scale/2 - footAnklePos}" origin_z="${footHeight/2}" width="${footWidth}" length="${footLength}" height="${footHeight}" mass="${footMass}" />
+	<xacro:create_box name="left_foot" origin_x="${footHeight*scale/2}" origin_y="${footLength*scale/2 - footAnklePos}" origin_z="0" r="0" p="${-PI/2}" y="0" width="${footWidth}" length="${footLength}" height="${footHeight}" mass="${footMass}" />
 	<!-- Left Lower Leg -->
-	<xacro:create_box name="left_lower_leg" origin_x="${-legDistFromCenter}" origin_y="0" origin_z="${lowerLegHeight/2 + footHeight - legAnklePos}" width="${lowerLegWidth}" length="${lowerLegLength}" height="${lowerLegHeight}" mass="${lowerLegMass}" />
+	<xacro:create_box name="left_lower_leg" origin_x="${lowerLegHeight*scale/2}" origin_y="0" origin_z="0" r="0" p="${-PI/2}" y="0" width="${lowerLegWidth}" length="${lowerLegLength}" height="${lowerLegHeight}" mass="${lowerLegMass}" />
 	<!-- Left Upper Leg -->
-	<xacro:create_box name="left_upper_leg" origin_x="${-legDistFromCenter}" origin_y="0" origin_z="${upperLegHeight/2 + footHeight - legAnklePos + lowerKneePos - upperKneePos}" width="${upperLegWidth}" length="${upperLegLength}" height="${upperLegHeight}" mass="${upperLegMass}" />
+	<xacro:create_box name="left_upper_leg" origin_x="${upperLegHeight*scale/2}" origin_y="0" origin_z="0" r="0" p="${-PI/2}" y="0" width="${upperLegWidth}" length="${upperLegLength}" height="${upperLegHeight}" mass="${upperLegMass}" />
 	<!--
 		Right Leg
 	-->
 	<!-- Right Foot -->
-	<xacro:create_box name="right_foot" origin_x="${legDistFromCenter}" origin_y="${footLength*scale/2 - footAnklePos}" origin_z="${footHeight/2}" width="${footWidth}" length="${footLength}" height="${footHeight}" mass="${footMass}" />
+	<xacro:create_box name="right_foot" origin_x="${footHeight*scale/2}" origin_y="${footLength*scale/2 - footAnklePos}" origin_z="0" r="0" p="${-PI/2}" y="0" width="${footWidth}" length="${footLength}" height="${footHeight}" mass="${footMass}" />
 	<!-- Right Lower Leg -->
-	<xacro:create_box name="right_lower_leg" origin_x="${legDistFromCenter}" origin_y="0" origin_z="${lowerLegHeight/2 + footHeight - legAnklePos}" width="${lowerLegWidth}" length="${lowerLegLength}" height="${lowerLegHeight}" mass="${lowerLegMass}" />
+	<xacro:create_box name="right_lower_leg" origin_x="${lowerLegHeight*scale/2}" origin_y="0" origin_z="0" r="0" p="${-PI/2}" y="0" width="${lowerLegWidth}" length="${lowerLegLength}" height="${lowerLegHeight}" mass="${lowerLegMass}" />
 	<!-- Right Upper Leg -->
-	<xacro:create_box name="right_upper_leg" origin_x="${legDistFromCenter}" origin_y="0" origin_z="${upperLegHeight/2 + footHeight - legAnklePos + lowerKneePos - upperKneePos}" width="${upperLegWidth}" length="${upperLegLength}" height="${upperLegHeight}" mass="${upperLegMass}" />
+	<xacro:create_box name="right_upper_leg" origin_x="${upperLegHeight*scale/2}" origin_y="0" origin_z="0" r="0" p="${-PI/2}" y="0" width="${upperLegWidth}" length="${upperLegLength}" height="${upperLegHeight}" mass="${upperLegMass}" />
 	<!--
 		Body
 	-->
-	<xacro:create_box name="body" origin_x="0" origin_y="${bodyWidth/2 - bodyHipWidth}" origin_z="${bodyHeight/2 + footHeight - legAnklePos + lowerKneePos - upperKneePos + legHipPos - bodyHipHeight}" width="${bodyWidth}" length="${bodyLength}" height="${bodyHeight}" mass="${bodyMass}" />
+	<xacro:create_box name="body" origin_x="0" origin_y="0" origin_z="${bodyHeight/2}" r="0" p="0" y="0" width="${bodyWidth}" length="${bodyLength}" height="${bodyHeight}" mass="${bodyMass}" />
+	<!--
+		Origin
+	-->
+	<link name="dacbot_origin"/>
 	<!--
 		Joints
 	-->
-	<!-- Used for fixing robot to Gazebo 'base_link' -->
-	<link name="world"/>
-	<joint name="world_left_foot" type="floating">
-		<parent link="world"/>
+	<joint name="dacbot" type="fixed">
+		<parent link="dacbot_origin"/>
+		<child link="body" />
+		<origin xyz="0 0 ${(bodyHeight*scale/2 + footHeight - legAnklePos + lowerKneePos - upperKneePos + legHipPos - bodyHipHeight)*2}" rpy="0 0 0"/>
+	</joint>
+	<joint name="left_hip" type="continuous">
+		<parent link="body"/>
+		<child link="left_upper_leg"/>
+		<origin xyz="${-legDistFromCenter} 0 0" rpy="0 ${PI/2} 0"/>
+		<axis xyz="0 0 1"/>
+		<dynamics damping="0.7"/>
+	</joint>
+	<joint name="left_knee" type="continuous">
+		<parent link="left_upper_leg"/>
+		<child link="left_lower_leg"/>
+		<origin xyz="${upperLegHeight} 0 0" rpy="0 0 0"/>
+		<axis xyz="0 0 1"/>
+		<dynamics damping="0.7"/>
+	</joint>
+	<joint name="left_ankle" type="continuous">
+		<parent link="left_lower_leg"/>
 		<child link="left_foot"/>
-	</joint>
-	<joint name="world_right_foot" type="floating">
-		<parent link="world"/>
+		<origin xyz="${lowerLegHeight} 0 0" rpy="0 0 0"/>
+		<axis xyz="0 0 1"/>
+		<dynamics damping="0.7"/>
+	</joint>
+	<joint name="right_hip" type="continuous">
+		<parent link="body"/>
+		<child link="right_upper_leg"/>
+		<origin xyz="${legDistFromCenter} 0 0" rpy="0 ${PI/2} 0"/>
+		<axis xyz="0 0 1"/>
+		<dynamics damping="0.7"/>
+	</joint>
+	<joint name="right_knee" type="continuous">
+		<parent link="right_upper_leg"/>
+		<child link="right_lower_leg"/>
+		<origin xyz="${upperLegHeight} 0 0" rpy="0 0 0"/>
+		<axis xyz="0 0 1"/>
+		<dynamics damping="0.7"/>
+	</joint>
+	<joint name="right_ankle" type="continuous">
+		<parent link="right_lower_leg"/>
 		<child link="right_foot"/>
-	</joint>
-	<joint name="left_ankle" type="continuous">
-		<parent link="left_foot"/>
-		<child link="left_lower_leg"/>
-		<origin xyz="${-legDistFromCenter} 0 ${footHeight/2}" rpy="0 0 0"/>
-		<axis xyz="1 0 0"/>
-		<dynamics damping="0.7"/>
-	</joint>
-	<joint name="left_knee" type="fixed">
-		<parent link="left_lower_leg"/>
-		<child link="left_upper_leg"/>
-		<origin xyz="${-legDistFromCenter} 0 0" rpy="0 0 0"/>
-		<axis xyz="1 0 0"/>
-		<dynamics damping="0.7"/>
-	</joint>
-	<joint name="left_hip" type="continuous">
-		<parent link="left_upper_leg"/>
-		<child link="body"/>
-		<origin xyz="${-legDistFromCenter} 0 0" rpy="0 0 0"/>
-		<axis xyz="1 0 0"/>
-		<dynamics damping="0.7"/>
-	</joint>
-	<joint name="right_ankle" type="continuous">
-		<parent link="right_foot"/>
-		<child link="right_lower_leg"/>
-		<origin xyz="${-legDistFromCenter} 0 ${footHeight/2}" rpy="0 0 0"/>
-		<axis xyz="1 0 0"/>
-		<dynamics damping="0.7"/>
-	</joint>
-	<joint name="right_knee" type="fixed">
-		<parent link="right_lower_leg"/>
-		<child link="right_upper_leg"/>
-		<origin xyz="${-legDistFromCenter} 0 0" rpy="0 0 0"/>
-		<axis xyz="1 0 0"/>
-		<dynamics damping="0.7"/>
-	</joint>
-	<joint name="right_hip" type="continuous">
-		<parent link="right_upper_leg"/>
-		<child link="body"/>
-		<origin xyz="${-legDistFromCenter} 0 0" rpy="0 0 0"/>
-		<axis xyz="1 0 0"/>
-		<dynamics damping="0.7"/>
-	</joint>
+		<origin xyz="${lowerLegHeight} 0 0" rpy="0 0 0"/>
+		<axis xyz="0 0 1"/>
+		<dynamics damping="0.7"/>
+	</joint>
+	<transmission name="left_hip_trans">
+		<type>transmission_interface/SimpleTransmission</type>
+			<joint name="left_hip">
+			<hardwareInterface>EffortJointInterface</hardwareInterface>
+		</joint>
+		<actuator name="left_hip_motor">
+			<hardwareInterface>EffortJointInterface</hardwareInterface>
+			<mechanicalReduction>1</mechanicalReduction>
+		</actuator>
+	</transmission>
+	<transmission name="left_knee_trans">
+		<type>transmission_interface/SimpleTransmission</type>
+			<joint name="left_knee">
+			<hardwareInterface>EffortJointInterface</hardwareInterface>
+		</joint>
+		<actuator name="left_knee_motor">
+			<hardwareInterface>EffortJointInterface</hardwareInterface>
+			<mechanicalReduction>1</mechanicalReduction>
+		</actuator>
+	</transmission>
+	<transmission name="left_ankle_trans">
+		<type>transmission_interface/SimpleTransmission</type>
+			<joint name="left_ankle">
+			<hardwareInterface>EffortJointInterface</hardwareInterface>
+		</joint>
+		<actuator name="left_ankle_motor">
+			<hardwareInterface>EffortJointInterface</hardwareInterface>
+			<mechanicalReduction>1</mechanicalReduction>
+		</actuator>
+	</transmission>
+	<transmission name="right_hip_trans">
+		<type>transmission_interface/SimpleTransmission</type>
+			<joint name="right_hip">
+			<hardwareInterface>EffortJointInterface</hardwareInterface>
+		</joint>
+		<actuator name="right_hip_motor">
+			<hardwareInterface>EffortJointInterface</hardwareInterface>
+			<mechanicalReduction>1</mechanicalReduction>
+		</actuator>
+	</transmission>
+	<transmission name="right_knee_trans">
+		<type>transmission_interface/SimpleTransmission</type>
+			<joint name="right_knee">
+			<hardwareInterface>EffortJointInterface</hardwareInterface>
+		</joint>
+		<actuator name="right_knee_motor">
+			<hardwareInterface>EffortJointInterface</hardwareInterface>
+			<mechanicalReduction>1</mechanicalReduction>
+		</actuator>
+	</transmission>
+	<transmission name="right_ankle_trans">
+		<type>transmission_interface/SimpleTransmission</type>
+			<joint name="right_ankle">
+			<hardwareInterface>EffortJointInterface</hardwareInterface>
+		</joint>
+		<actuator name="right_ankle_motor">
+			<hardwareInterface>EffortJointInterface</hardwareInterface>
+			<mechanicalReduction>1</mechanicalReduction>
+		</actuator>
+	</transmission>
 </robot>

Commit message: risen a bit the robot in gazebo

File: src/dacbot_description/urdf/dacbot.urdf (robot description, URDF)
Before this commit: robot dacbot, 8 links, 7 joints
Links:
- removed link dacbot_origin
Joints:
- removed joint dacbot

File: src/dacbot_description/urdf/dacbot.xacro (robot description, xacro)
@@ -104,15 +104,6 @@
 	<xacro:create_box name="body" origin_x="0" origin_y="0" origin_z="${bodyHeight/2}" r="0" p="0" y="0" width="${bodyWidth}" length="${bodyLength}" height="${bodyHeight}" mass="${bodyMass}" />
 	<!--
-		Origin
-	-->
-	<link name="dacbot_origin"/>
-	<!--
 		Joints
 	-->
-	<joint name="dacbot" type="fixed">
-		<parent link="dacbot_origin"/>
-		<child link="body" />
-		<origin xyz="0 0 ${(bodyHeight*scale/2 + footHeight - legAnklePos + lowerKneePos - upperKneePos + legHipPos - bodyHipHeight)*2}" rpy="0 0 0"/>
-	</joint>
 	<joint name="left_hip" type="continuous">
 		<parent link="body"/>

Commit message: fixed scale problems. The problem with gazebo its due to the moemnts of inertia are really small

File: src/dacbot_description/urdf/dacbot.urdf (robot description, URDF)
Before this commit: robot dacbot, 7 links, 6 joints
Links:
- link body: mass 0.45 -> 2.25; geometry collision box size=0.425 0.4 0.325; visual box size=0.425 0.4 0.325
- link left_foot: mass 0.01 -> 0.05; geometry collision box size=0.075 0.25 0.04; visual box size=0.075 0.25 0.04
- link left_lower_leg: mass 0.08 -> 0.4; geometry collision box size=0.075 0.075 0.625; visual box size=0.075 0.075 0.625
- link left_upper_leg: mass 0.2 -> 1.0; geometry collision box size=0.075 0.075 0.71; visual box size=0.075 0.075 0.71
- link right_foot: mass 0.01 -> 0.05; geometry collision box size=0.075 0.25 0.04; visual box size=0.075 0.25 0.04
- link right_lower_leg: mass 0.08 -> 0.4; geometry collision box size=0.075 0.075 0.625; visual box size=0.075 0.075 0.625
- link right_upper_leg: mass 0.2 -> 1.0; geometry collision box size=0.075 0.075 0.71; visual box size=0.075 0.075 0.71
Joints:
- joint left_ankle: origin xyz=0.125 0 0 rpy=0 0 0 -> xyz=0.625 0 0 rpy=0 0 0
- joint left_hip: origin xyz=-0.015 0 0 rpy=0 1.57079632679 0 -> xyz=-0.075 0 0 rpy=0 1.57079632679 0
- joint left_knee: origin xyz=0.142 0 0 rpy=0 0 0 -> xyz=0.71 0 0 rpy=0 0 0
- joint right_ankle: origin xyz=0.125 0 0 rpy=0 0 0 -> xyz=0.625 0 0 rpy=0 0 0
- joint right_hip: origin xyz=0.015 0 0 rpy=0 1.57079632679 0 -> xyz=0.075 0 0 rpy=0 1.57079632679 0
- joint right_knee: origin xyz=0.142 0 0 rpy=0 0 0 -> xyz=0.71 0 0 rpy=0 0 0

File: src/dacbot_description/urdf/dacbot.xacro (robot description, xacro)
@@ -8,39 +8,39 @@
 		Height = Z axis
 	-->
-	<xacro:property name="scale" value="1" />
-	<xacro:property name="bodyWidth" value="0.085" />
-	<xacro:property name="bodyLength" value="0.08" />
-	<xacro:property name="bodyHeight" value="0.065" />
-	<xacro:property name="bodyMass" value="0.45" />
-	<xacro:property name="weightWidth" value="0.05" />
-	<xacro:property name="weightLength" value="0.07" />
-	<xacro:property name="weightHeight" value="0.025" />
-	<xacro:property name="weightMass" value="0.50" />
-	<xacro:property name="upperLegWidth" value="0.015" />
-	<xacro:property name="upperLegLength" value="0.015" />
-	<xacro:property name="upperLegHeight" value="0.142" />
-	<xacro:property name="upperLegMass" value="0.2" />
-	<xacro:property name="lowerLegWidth" value="0.015" />
-	<xacro:property name="lowerLegLength" value="0.015" />
-	<xacro:property name="lowerLegHeight" value="0.125" />
-	<xacro:property name="lowerLegMass" value="0.08" />
-	<xacro:property name="footWidth" value="0.015" />
-	<xacro:property name="footLength" value="0.050" />
-	<xacro:property name="footHeight" value="0.008" />
-	<xacro:property name="footMass" value="0.01" />
-	<xacro:property name="legDistFromCenter" value="0.015" />
-	<xacro:property name="footAnklePos" value="0.015" />
-	<xacro:property name="legAnklePos" value="0" />
-	<xacro:property name="lowerKneePos" value="0.12" />
-	<xacro:property name="upperKneePos" value="0.02" />
-	<xacro:property name="legHipPos" value="0.132" />
-	<xacro:property name="bodyHipHeight" value="0.01" />
-	<xacro:property name="bodyHipWidth" value="0.025" />
-	<xacro:property name="massJointBodyDepth" value="0.07" />
-	<xacro:property name="massJointBodyHeight" value="0.055" />
-	<xacro:property name="massJointMassDepth" value="0.065" />
-	<xacro:property name="massJointMassHeigth" value="0.007" />
-	<xacro:property name="armLength" value="0.6" />
-	<xacro:property name="armOffset" value="0.025" />
+	<xacro:property name="scale" value="5" />
+	<xacro:property name="bodyWidth" value="${0.085*scale}" />
+	<xacro:property name="bodyLength" value="${0.08*scale}" />
+	<xacro:property name="bodyHeight" value="${0.065*scale}" />
+	<xacro:property name="bodyMass" value="${0.45*scale}" />
+	<xacro:property name="weightWidth" value="${0.05*scale}" />
+	<xacro:property name="weightLength" value="${0.07*scale}" />
+	<xacro:property name="weightHeight" value="${0.025*scale}" />
+	<xacro:property name="weightMass" value="${0.50*scale}" />
+	<xacro:property name="upperLegWidth" value="${0.015*scale}" />
+	<xacro:property name="upperLegLength" value="${0.015*scale}" />
+	<xacro:property name="upperLegHeight" value="${0.142*scale}" />
+	<xacro:property name="upperLegMass" value="${0.2*scale}" />
+	<xacro:property name="lowerLegWidth" value="${0.015*scale}" />
+	<xacro:property name="lowerLegLength" value="${0.015*scale}" />
+	<xacro:property name="lowerLegHeight" value="${0.125*scale}" />
+	<xacro:property name="lowerLegMass" value="${0.08*scale}" />
+	<xacro:property name="footWidth" value="${0.015*scale}" />
+	<xacro:property name="footLength" value="${0.050*scale}" />
+	<xacro:property name="footHeight" value="${0.008*scale}" />
+	<xacro:property name="footMass" value="${0.01*scale}" />
+	<xacro:property name="legDistFromCenter" value="${0.015*scale}" />
+	<xacro:property name="footAnklePos" value="${0.015*scale}" />
+	<xacro:property name="legAnklePos" value="${0*scale}" />
+	<xacro:property name="lowerKneePos" value="${0.12*scale}" />
+	<xacro:property name="upperKneePos" value="${0.02*scale}" />
+	<xacro:property name="legHipPos" value="${0.132*scale}" />
+	<xacro:property name="bodyHipHeight" value="${0.01*scale}" />
+	<xacro:property name="bodyHipWidth" value="${0.025*scale}" />
+	<xacro:property name="massJointBodyDepth" value="${0.07*scale}" />
+	<xacro:property name="massJointBodyHeight" value="${0.055*scale}" />
+	<xacro:property name="massJointMassDepth" value="${0.065*scale}" />
+	<xacro:property name="massJointMassHeigth" value="${0.007*scale}" />
+	<xacro:property name="armLength" value="${0.6*scale}" />
+	<xacro:property name="armOffset" value="${0.025*scale}" />
 	<!-- Import Gazebo customizations and colors-->
 	<xacro:include filename="$(find dacbot_description)/urdf/dacbot.gazebo" />
@@ -57,5 +57,5 @@
 				<origin xyz="${origin_x} ${origin_y} ${origin_z}" rpy="${r} ${p} ${y}"/>
 				<geometry>
-					<box size="${width*scale} ${length*scale} ${height*scale}" />
+					<box size="${width} ${length} ${height}" />
 				</geometry>
 			</collision>
@@ -63,5 +63,5 @@
 				<origin xyz="${origin_x} ${origin_y} ${origin_z}" rpy="${r} ${p} ${y}"/>
 				<geometry>
-					<box size="${width*scale} ${length*scale} ${height*scale}" />
+					<box size="${width} ${length} ${height}" />
 				</geometry>
 				<material name="orange"/>
@@ -85,18 +85,18 @@
 	-->
 	<!-- Left Foot -->
-	<xacro:create_box name="left_foot" origin_x="${footHeight*scale/2}" origin_y="${footLength*scale/2 - footAnklePos}" origin_z="0" r="0" p="${-PI/2}" y="0" width="${footWidth}" length="${footLength}" height="${footHeight}" mass="${footMass}" />
+	<xacro:create_box name="left_foot" origin_x="${footHeight/2}" origin_y="${footLength/2 - footAnklePos}" origin_z="0" r="0" p="${-PI/2}" y="0" width="${footWidth}" length="${footLength}" height="${footHeight}" mass="${footMass}" />
 	<!-- Left Lower Leg -->
-	<xacro:create_box name="left_lower_leg" origin_x="${lowerLegHeight*scale/2}" origin_y="0" origin_z="0" r="0" p="${-PI/2}" y="0" width="${lowerLegWidth}" length="${lowerLegLength}" height="${lowerLegHeight}" mass="${lowerLegMass}" />
+	<xacro:create_box name="left_lower_leg" origin_x="${lowerLegHeight/2}" origin_y="0" origin_z="0" r="0" p="${-PI/2}" y="0" width="${lowerLegWidth}" length="${lowerLegLength}" height="${lowerLegHeight}" mass="${lowerLegMass}" />
 	<!-- Left Upper Leg -->
-	<xacro:create_box name="left_upper_leg" origin_x="${upperLegHeight*scale/2}" origin_y="0" origin_z="0" r="0" p="${-PI/2}" y="0" width="${upperLegWidth}" length="${upperLegLength}" height="${upperLegHeight}" mass="${upperLegMass}" />
+	<xacro:create_box name="left_upper_leg" origin_x="${upperLegHeight/2}" origin_y="0" origin_z="0" r="0" p="${-PI/2}" y="0" width="${upperLegWidth}" length="${upperLegLength}" height="${upperLegHeight}" mass="${upperLegMass}" />
 	<!--
 		Right Leg
 	-->
 	<!-- Right Foot -->
-	<xacro:create_box name="right_foot" origin_x="${footHeight*scale/2}" origin_y="${footLength*scale/2 - footAnklePos}" origin_z="0" r="0" p="${-PI/2}" y="0" width="${footWidth}" length="${footLength}" height="${footHeight}" mass="${footMass}" />
+	<xacro:create_box name="right_foot" origin_x="${footHeight/2}" origin_y="${footLength/2 - footAnklePos}" origin_z="0" r="0" p="${-PI/2}" y="0" width="${footWidth}" length="${footLength}" height="${footHeight}" mass="${footMass}" />
 	<!-- Right Lower Leg -->
-	<xacro:create_box name="right_lower_leg" origin_x="${lowerLegHeight*scale/2}" origin_y="0" origin_z="0" r="0" p="${-PI/2}" y="0" width="${lowerLegWidth}" length="${lowerLegLength}" height="${lowerLegHeight}" mass="${lowerLegMass}" />
+	<xacro:create_box name="right_lower_leg" origin_x="${lowerLegHeight/2}" origin_y="0" origin_z="0" r="0" p="${-PI/2}" y="0" width="${lowerLegWidth}" length="${lowerLegLength}" height="${lowerLegHeight}" mass="${lowerLegMass}" />
 	<!-- Right Upper Leg -->
-	<xacro:create_box name="right_upper_leg" origin_x="${upperLegHeight*scale/2}" origin_y="0" origin_z="0" r="0" p="${-PI/2}" y="0" width="${upperLegWidth}" length="${upperLegLength}" height="${upperLegHeight}" mass="${upperLegMass}" />
+	<xacro:create_box name="right_upper_leg" origin_x="${upperLegHeight/2}" origin_y="0" origin_z="0" r="0" p="${-PI/2}" y="0" width="${upperLegWidth}" length="${upperLegLength}" height="${upperLegHeight}" mass="${upperLegMass}" />
 	<!--
 		Body
