Commit message: Set a minimum intertia value to avoid problems in gazebo

File: src/dacbot_description/urdf/dacbot.urdf (robot description, URDF)
Before this commit: robot dacbot, 7 links, 6 joints
Links:
- link body: mass 2.25 -> 0.45; geometry collision box size=0.085 0.08 0.065; visual box size=0.085 0.08 0.065
- link left_foot: mass 0.05 -> 0.01; geometry collision box size=0.015 0.05 0.008; visual box size=0.015 0.05 0.008
- link left_lower_leg: mass 0.4 -> 0.08; geometry collision box size=0.015 0.015 0.125; visual box size=0.015 0.015 0.125
- link left_upper_leg: mass 1.0 -> 0.2; geometry collision box size=0.015 0.015 0.142; visual box size=0.015 0.015 0.142
- link right_foot: mass 0.05 -> 0.01; geometry collision box size=0.015 0.05 0.008; visual box size=0.015 0.05 0.008
- link right_lower_leg: mass 0.4 -> 0.08; geometry collision box size=0.015 0.015 0.125; visual box size=0.015 0.015 0.125
- link right_upper_leg: mass 1.0 -> 0.2; geometry collision box size=0.015 0.015 0.142; visual box size=0.015 0.015 0.142
Joints:
- joint left_ankle: origin xyz=0.625 0 0 rpy=0 0 0 -> xyz=0.125 0 0 rpy=0 0 0
- joint left_hip: origin xyz=-0.075 0 0 rpy=0 1.57079632679 0 -> xyz=-0.015 0 0 rpy=0 1.57079632679 0
- joint left_knee: origin xyz=0.71 0 0 rpy=0 0 0 -> xyz=0.142 0 0 rpy=0 0 0
- joint right_ankle: origin xyz=0.625 0 0 rpy=0 0 0 -> xyz=0.125 0 0 rpy=0 0 0
- joint right_hip: origin xyz=0.075 0 0 rpy=0 1.57079632679 0 -> xyz=0.015 0 0 rpy=0 1.57079632679 0
- joint right_knee: origin xyz=0.71 0 0 rpy=0 0 0 -> xyz=0.142 0 0 rpy=0 0 0

File: src/dacbot_description/urdf/dacbot.xacro (robot description, xacro)
@@ -8,5 +8,5 @@
 		Height = Z axis
 	-->
-	<xacro:property name="scale" value="5" />
+	<xacro:property name="scale" value="1" />
 	<xacro:property name="bodyWidth" value="${0.085*scale}" />
 	<xacro:property name="bodyLength" value="${0.08*scale}" />
@@ -53,4 +53,18 @@
 	 -->
 	<xacro:macro name="create_box" params="name origin_x origin_y origin_z r p y width length height mass">
+		<!-- Set the minimum intertia as 0.01 -->
+		<xacro:property name="ixx" value="0.01" />
+		<xacro:if value="${mass / 12.0 * (length*length + height*height) > 0.01}">
+			<xacro:property name="ixx" value="${mass / 12.0 * (length*length + height*height)}" />
+		</xacro:if>
+		<xacro:property name="iyy" value="0.01" />
+		<xacro:if value="${mass / 12.0 * (length*length + height*height) > 0.01}">
+			<xacro:property name="iyy" value="${mass / 12.0 * (length*length + height*height)}" />
+		</xacro:if>
+		<xacro:property name="izz" value="0.01" />
+		<xacro:if value="${mass / 12.0 * (length*length + height*height) > 0.01}">
+			<xacro:property name="izz" value="${mass / 12.0 * (length*length + height*height)}" />
+		</xacro:if>
+		<!-- Creates the link -->
 		<link name="${name}">
 			<collision>
@@ -71,7 +85,7 @@
 				<mass value="${mass}"/>
 				<inertia
-					ixx="${mass / 12.0 * (length*length + height*height)*scale*scale}" ixy="0.0" ixz="0.0"
-					iyy="${mass / 12.0 * (height*height + width*width)*scale*scale}" iyz="0.0"
-					izz="${mass / 12.0 * (width*width + length*length)*scale*scale}"/>
+					ixx="${ixx}" ixy="0.0" ixz="0.0"
+					iyy="${iyy}" iyz="0.0"
+					izz="${izz}"/>
 			</inertial>
 		</link>

Commit message: Body fixed

File: src/dacbot_description/urdf/dacbot.urdf (robot description, URDF)
Before this commit: robot dacbot, 7 links, 6 joints
Links:
- added link world
Joints:
- added joint fixed: type fixed, parent world, child body, origin xyz=0 0 0.3025 rpy=0 0 0

File: src/dacbot_description/urdf/dacbot.xacro (robot description, xacro)
@@ -121,4 +121,10 @@
 		Joints
 	-->
+  <link name="world"/>
+  <joint name="fixed" type="fixed">
+    <parent link="world"/>
+    <child link="body"/>
+    <origin xyz="0 0 ${(footHeight + lowerLegHeight + upperLegHeight)*1.1}" rpy="0 0 0"/>
+  </joint>
 	<joint name="left_hip" type="continuous">
 		<parent link="body"/>

Commit message: added rotational robot holder

File: src/dacbot_description/urdf/dacbot.urdf (robot description, URDF)
Before this commit: robot dacbot, 8 links, 7 joints
Links:
- added link rotational_robot_holder_base, mass 10; collision cylinder length=0.275 radius=0.2; visual cylinder length=0.275 radius=0.2
- added link rotational_robot_holder_holder, mass 0.01; collision cylinder length=2 radius=0.01; visual cylinder length=2 radius=0.01
Joints:
- removed joint fixed
- added joint rotational_robot_holder_base_to_world: type fixed, parent world, child rotational_robot_holder_base, origin xyz=0 0 0.1375 rpy=0 0 0
- added joint rotational_robot_holder_joint: type continuous, parent rotational_robot_holder_base, child rotational_robot_holder_holder, origin xyz=0 0 0.1375 rpy=0 0 0, axis 0 0 1
- added joint rotational_robot_holder_to_rotot: type continuous, parent rotational_robot_holder_holder, child body, origin xyz=2 0 0 rpy=0 0 0, axis 1 0 0

File: src/dacbot_description/urdf/dacbot.xacro (robot description, xacro)
@@ -124,9 +124,9 @@
 	-->
   <link name="world"/>
-  <joint name="fixed" type="fixed">
+<!--   <joint name="fixed" type="fixed">
     <parent link="world"/>
     <child link="body"/>
     <origin xyz="0 0 ${(footHeight + lowerLegHeight + upperLegHeight)*1.1}" rpy="0 0 0"/>
-  </joint>
+  </joint>  -->
 	<joint name="left_hip" type="continuous">
 		<parent link="body"/>
@@ -231,3 +231,9 @@
 		</actuator>
 	</transmission>
+	<!-- Rotational robot holder -->
+	<xacro:property name="rotational_robot_holder_base_radius" value="${0.2*scale}" />
+  <xacro:property name="rotational_robot_holder_base_length" value="${(footHeight + lowerLegHeight + upperLegHeight)*scale}" />
+  <xacro:property name="rotational_robot_holder_holder_radius" value="${0.01*scale}" />
+  <xacro:property name="rotational_robot_holder_holder_length" value="${2*scale}" />
+	<xacro:include filename="$(find gazebo_resources)/models/rotational_robot_holder/urdf/rotational_robot_holder.xacro" />
 </robot>

Commit message: Added feet contact sensors making use of the bumper plugin

File: src/dacbot_description/urdf/dacbot.urdf (robot description, URDF)
Before this commit: robot dacbot, 10 links, 9 joints
Joints:
- joint rotational_robot_holder_to_rotot: axis 1 0 0 -> (none); type continuous -> fixed

File: src/dacbot_description/urdf/dacbot.xacro (robot description, xacro)
@@ -3,4 +3,7 @@
 	<!-- Constants -->
 	<xacro:property name="PI" value="3.1415926535897931"/>
+	<!-- ROS -->
+	<xacro:property name="update_rate" value="2"/>
+	<xacro:property name="robot_name" value="dacbot"/>
 	<!-- Robot configuration: Transmission -->
 	<xacro:property name="maxRealMotorTorque" value="1.0787315"/> <!-- In N*m -->
@@ -53,5 +56,5 @@
 	 -->
 	 <!-- Box Macro!
-	<xacro:create_box name="" origin_x="" origin_y="" origin_z="" r="" p="" y="" width="" length="" height="" mass="" />
+	<xacro:create_box name="" origin_x="" origin_y="" origin_z="" r="" p="" y="" width="" length="" height="" mass=""/>
 	 -->
 	<xacro:macro name="create_box" params="name origin_x origin_y origin_z r p y width length height mass">
@@ -102,22 +105,22 @@
 	-->
 	<!-- Left Foot -->
-	<xacro:create_box name="left_foot" origin_x="${footHeight/2}" origin_y="${footLength/2 - footAnklePos}" origin_z="0" r="0" p="${-PI/2}" y="0" width="${footWidth}" length="${footLength}" height="${footHeight}" mass="${footMass}" />
+	<xacro:create_box name="left_foot" origin_x="${footHeight/2}" origin_y="${footLength/2 - footAnklePos}" origin_z="0" r="0" p="${-PI/2}" y="0" width="${footWidth}" length="${footLength}" height="${footHeight}" mass="${footMass}"  />
 	<!-- Left Lower Leg -->
-	<xacro:create_box name="left_lower_leg" origin_x="${lowerLegHeight/2}" origin_y="0" origin_z="0" r="0" p="${-PI/2}" y="0" width="${lowerLegWidth}" length="${lowerLegLength}" height="${lowerLegHeight}" mass="${lowerLegMass}" />
+	<xacro:create_box name="left_lower_leg" origin_x="${lowerLegHeight/2}" origin_y="0" origin_z="0" r="0" p="${-PI/2}" y="0" width="${lowerLegWidth}" length="${lowerLegLength}" height="${lowerLegHeight}" mass="${lowerLegMass}"  />
 	<!-- Left Upper Leg -->
-	<xacro:create_box name="left_upper_leg" origin_x="${upperLegHeight/2}" origin_y="0" origin_z="0" r="0" p="${-PI/2}" y="0" width="${upperLegWidth}" length="${upperLegLength}" height="${upperLegHeight}" mass="${upperLegMass}" />
+	<xacro:create_box name="left_upper_leg" origin_x="${upperLegHeight/2}" origin_y="0" origin_z="0" r="0" p="${-PI/2}" y="0" width="${upperLegWidth}" length="${upperLegLength}" height="${upperLegHeight}" mass="${upperLegMass}"   />
 	<!--
 		Right Leg
 	-->
 	<!-- Right Foot -->
-	<xacro:create_box name="right_foot" origin_x="${footHeight/2}" origin_y="${footLength/2 - footAnklePos}" origin_z="0" r="0" p="${-PI/2}" y="0" width="${footWidth}" length="${footLength}" height="${footHeight}" mass="${footMass}" />
+	<xacro:create_box name="right_foot" origin_x="${footHeight/2}" origin_y="${footLength/2 - footAnklePos}" origin_z="0" r="0" p="${-PI/2}" y="0" width="${footWidth}" length="${footLength}" height="${footHeight}" mass="${footMass}"   />
 	<!-- Right Lower Leg -->
-	<xacro:create_box name="right_lower_leg" origin_x="${lowerLegHeight/2}" origin_y="0" origin_z="0" r="0" p="${-PI/2}" y="0" width="${lowerLegWidth}" length="${lowerLegLength}" height="${lowerLegHeight}" mass="${lowerLegMass}" />
+	<xacro:create_box name="right_lower_leg" origin_x="${lowerLegHeight/2}" origin_y="0" origin_z="0" r="0" p="${-PI/2}" y="0" width="${lowerLegWidth}" length="${lowerLegLength}" height="${lowerLegHeight}" mass="${lowerLegMass}"   />
 	<!-- Right Upper Leg -->
-	<xacro:create_box name="right_upper_leg" origin_x="${upperLegHeight/2}" origin_y="0" origin_z="0" r="0" p="${-PI/2}" y="0" width="${upperLegWidth}" length="${upperLegLength}" height="${upperLegHeight}" mass="${upperLegMass}" />
+	<xacro:create_box name="right_upper_leg" origin_x="${upperLegHeight/2}" origin_y="0" origin_z="0" r="0" p="${-PI/2}" y="0" width="${upperLegWidth}" length="${upperLegLength}" height="${upperLegHeight}" mass="${upperLegMass}"   />
 	<!--
 		Body
 	-->
-	<xacro:create_box name="body" origin_x="0" origin_y="0" origin_z="${bodyHeight/2}" r="0" p="0" y="0" width="${bodyWidth}" length="${bodyLength}" height="${bodyHeight}" mass="${bodyMass}" />
+	<xacro:create_box name="body" origin_x="0" origin_y="0" origin_z="${bodyHeight/2}" r="0" p="0" y="0" width="${bodyWidth}" length="${bodyLength}" height="${bodyHeight}" mass="${bodyMass}"  />
 	<!--
 		Joints

Commit message: updated parameters

File: src/dacbot_description/urdf/dacbot.urdf (robot description, URDF)
Before this commit: robot dacbot, 10 links, 9 joints
Links:
- added link rotational_robot_holder_virtual, mass 0.01; collision sphere radius=0.01; visual sphere radius=0.01
- link rotational_robot_holder_base: geometry collision cylinder length=0.375 radius=0.2; visual cylinder length=0.375 radius=0.2
Joints:
- added joint rotational_robot_holder_virtual_to_holder: type fixed, parent rotational_robot_holder_base, child rotational_robot_holder_virtual
- joint left_ankle: limit (none) -> lower=0 upper=0 effort=10 velocity=10; type continuous -> revolute
- joint left_hip: limit (none) -> lower=-0.523598775598 upper=0.523598775598 effort=10 velocity=10; type continuous -> revolute
- joint left_knee: limit (none) -> lower=-2.61799387799 upper=0.0 effort=10 velocity=10; type continuous -> revolute
- joint right_ankle: limit (none) -> lower=0 upper=0 effort=10 velocity=10; type continuous -> revolute
- joint right_hip: limit (none) -> lower=-0.523598775598 upper=0.523598775598 effort=10 velocity=10; type continuous -> revolute
- joint right_knee: limit (none) -> lower=-2.61799387799 upper=0.0 effort=10 velocity=10; type continuous -> revolute
- joint rotational_robot_holder_base_to_world: origin xyz=0 0 0.1375 rpy=0 0 0 -> xyz=0 0 0.1875 rpy=0 0 0
- joint rotational_robot_holder_joint: axis 0 0 1 -> (none); origin xyz=0 0 0.1375 rpy=0 0 0 -> xyz=0 0 0.1875 rpy=0 0 0; parent rotational_robot_holder_base -> rotational_robot_holder_virtual; type continuous -> fixed
- joint rotational_robot_holder_to_rotot: axis (none) -> 0 0 1; limit (none) -> lower=0 upper=1 effort=30 velocity=1.0; origin xyz=2 0 0 rpy=0 0 0 -> xyz=2.0425 0 0 rpy=0 0 0

File: src/dacbot_description/urdf/dacbot.xacro (robot description, xacro)
@@ -18,5 +18,4 @@
   <xacro:property name="scale" value="1" />
   <xacro:property name="minimum_intertia" value="0.002" /> <!-- <0.001 doesn't work -->
-  <xacro:property name="damping" value="0.8"/>
 	<xacro:property name="bodyWidth" value="${0.085*scale}" />
 	<xacro:property name="bodyLength" value="${0.08*scale}" />
@@ -31,6 +30,6 @@
 	<xacro:property name="upperLegHeight" value="${0.142*scale}" />
 	<xacro:property name="upperLegMass" value="${0.2*scale}" />
-  <xacro:property name="upperLegLimitUpperPosition" value="70" />
-  <xacro:property name="upperLegLimitLowerPosition" value="-70" />
+  <xacro:property name="upperLegLimitUpperPosition" value="30" />
+  <xacro:property name="upperLegLimitLowerPosition" value="-30" />
   <xacro:property name="upperLegLimitVelocity" value="10" />
   <xacro:property name="upperLegLimitEffort" value="10" />
@@ -41,5 +40,5 @@
 	<xacro:property name="lowerLegMass" value="${0.08*scale}" />
   <xacro:property name="lowerLegLimitUpperPosition" value="0" />
-  <xacro:property name="lowerLegLimitLowerPosition" value="150" />
+  <xacro:property name="lowerLegLimitLowerPosition" value="-150" />
   <xacro:property name="lowerLegLimitVelocity" value="10" />
   <xacro:property name="lowerLegLimitEffort" value="10" />
