Commit message: Updated to use macros

File: src/dacbot_description/urdf/dacbot.xacro (robot description, xacro)
@@ -17,9 +17,11 @@
 	<xacro:property name="weightHeight" value="0.025" />
 	<xacro:property name="weightMass" value="0.50" />
-	<xacro:property name="upperLegLength" value="0.0142" />
-	<xacro:property name="upperLegThickness" value="0.015" />
+	<xacro:property name="upperLegWidth" value="0.015" />
+	<xacro:property name="upperLegLength" value="0.015" />
+	<xacro:property name="upperLegHeight" value="0.142" />
 	<xacro:property name="upperLegMass" value="0.2" />
-	<xacro:property name="lowerLegLength" value="0.0125" />
-	<xacro:property name="lowerLegThickness" value="0.015" />
+	<xacro:property name="lowerLegWidth" value="0.015" />
+	<xacro:property name="lowerLegLength" value="0.015" />
+	<xacro:property name="lowerLegHeight" value="0.125" />
 	<xacro:property name="lowerLegMass" value="0.08" />
 	<xacro:property name="footWidth" value="0.015" />
@@ -50,61 +52,73 @@
 		<child link="left_foot"/>
 	</joint>
-	<joint name="fixed_right" type="fixed">
-		<parent link="world"/>
-		<child link="right_foot"/>
-	</joint>
+	<!--
+		Macros
+	 -->
+	 <!-- Box Macro!
+	<xacro:box name="" origin_x="" origin_y="" origin_z="" width="" length="" height="" mass="" />
+	 -->
+	<xacro:macro name="create_box" params="name origin_x origin_y origin_z width length height mass">
+		<link name="${name}">
+			<collision>
+				<origin xyz="${origin_x} ${origin_y} ${origin_z}" rpy="0 0 0"/>
+				<geometry>
+					<box size="${width*scale} ${length*scale} ${height*scale}" />
+				</geometry>
+			</collision>
+			<visual>
+				<origin xyz="${origin_x} ${origin_y} ${origin_z}" rpy="0 0 0"/>
+				<geometry>
+					<box size="${width*scale} ${length*scale} ${height*scale}" />
+				</geometry>
+				<material name="orange"/>
+			</visual>
+			<inertial>
+				<origin xyz="${origin_x} ${origin_y} ${origin_z}" rpy="0 0 0"/>
+				<mass value="${mass}"/>
+				<inertia
+					ixx="${mass / 12.0 * (length*length + height*height)*scale*scale}" ixy="0.0" ixz="0.0"
+					iyy="${mass / 12.0 * (height*height + width*width)*scale*scale}" iyz="0.0"
+					izz="${mass / 12.0 * (width*width + length*length)*scale*scale}"/>
+			</inertial>
+		</link>
+	</xacro:macro>
 	<!--
 		Left Leg
 	-->
 	<!-- Left Foot -->
-	<link name="left_foot">
+	<xacro:property name="var" value="1"/>
+	<xacro:create_box name="left_foot" origin_x="${var}" origin_y="${footLength*scale/2 - footAnklePos}" origin_z="${footHeight/2}" width="${footWidth}" length="${footLength}" height="${footHeight}" mass="${footMass}" />
+	<!-- Left Foot -->
+	<xacro:property name="var" value"${var} + 1"/>
+	<xacro:create_box name="left_lower_leg" origin_x="${var}" origin_y="${footLength*scale/2 - footAnklePos}" origin_z="${footHeight/2}" width="${footWidth}" length="${footLength}" height="${footHeight}" mass="${footMass}" />
+	<!-- Left Lower Leg -->
+	<!--
+	<link name="left_lower_leg">
 		<collision>
-			<origin xyz="${-bodyWidth/2} 0 ${footHeight/2}" rpy="0 0 0"/>
+			<origin xyz="${-legDistFromCenter} 0 ${footHeight + lowerLegHeight*scale/2}" rpy="0 0 0"/>
 			<geometry>
-				<box size="${footWidth*scale} ${footLength*scale} ${footHeight*scale}" />
+				<box size="${lowerLegWidth*scale} ${lowerLegLength*scale} ${lowerLegHeight*scale}" />
 			</geometry>
 		</collision>
 		<visual>
-			<origin xyz="${-bodyWidth/2} 0 ${footHeight/2}" rpy="0 0 0"/>
+			<origin xyz="${-bodyWidth/2} 0 ${footHeight + lowerLegHeight/2}" rpy="0 0 0"/>
 			<geometry>
-				<box size="${footWidth*scale} ${footLength*scale} ${footHeight*scale}" />
+				<box size="${lowerLegWidth*scale} ${lowerLegLength*scale} ${lowerLegHeight*scale}" />
 			</geometry>
 			<material name="orange"/>
 		</visual>
 		<inertial>
-			<origin xyz="${-bodyWidth/2} 0 ${footHeight/2}" rpy="0 0 0"/>
+			<origin xyz="${-bodyWidth/2} 0 ${footHeight + lowerLegHeight/2}" rpy="0 0 0"/>
 			<mass value="${footMass}"/>
 			<inertia
-				ixx="${footMass / 12.0 * (footWidth*footWidth + footHeight*footHeight)}" ixy="0.0" ixz="0.0"
-				iyy="${footMass / 12.0 * (footHeight*footHeight + footWidth*footWidth)}" iyz="0.0"
-				izz="${footMass / 12.0 * (footWidth*footWidth + footWidth*footWidth)}"/>
+				ixx="${footMass / 12.0 * (lowerLegWidth*lowerLegWidth + lowerLegHeight*lowerLegHeight)}" ixy="0.0" ixz="0.0"
+				iyy="${footMass / 12.0 * (lowerLegHeight*lowerLegHeight + lowerLegWidth*lowerLegWidth)}" iyz="0.0"
+				izz="${footMass / 12.0 * (lowerLegWidth*lowerLegWidth + lowerLegWidth*lowerLegWidth)}"/>
 		</inertial>
 	</link>
-	<!--
-		Right Leg
-	-->
-	<!-- Right Foot -->
-	<link name="right_foot">
-		<collision>
-			<origin xyz="${bodyWidth/2} 0 ${footHeight/2}" rpy="0 0 0"/>
-			<geometry>
-				<box size="${footWidth*scale} ${footLength*scale} ${footHeight*scale}" />
-			</geometry>
-		</collision>
-		<visual>
-			<origin xyz="${bodyWidth/2} 0 ${footHeight/2}" rpy="0 0 0"/>
-			<geometry>
-				<box size="${footWidth*scale} ${footLength*scale} ${footHeight*scale}" />
-			</geometry>
-			<material name="orange"/>
-		</visual>
-		<inertial>
-			<origin xyz="${bodyWidth/2} 0 ${footHeight/2}" rpy="0 0 0"/>
-			<mass value="${footMass}"/>
-			<inertia
-				ixx="${footMass / 12.0 * (footWidth*footWidth + footHeight*footHeight)}" ixy="0.0" ixz="0.0"
-				iyy="${footMass / 12.0 * (footHeight*footHeight + footWidth*footWidth)}" iyz="0.0"
-				izz="${footMass / 12.0 * (footWidth*footWidth + footWidth*footWidth)}"/>
-		</inertial>
-	</link>
+	<joint name="left_ankle" type="fixed">
+		<parent link="left_foot"/>
+		<child link="left_lower_leg"/>
+	</joint>
+-->
 </robot>

Commit message: all parts added and compiles, but doesnt work yet!

File: src/dacbot_description/urdf/dacbot.xacro (robot description, xacro)
@@ -32,9 +32,9 @@
 	<xacro:property name="footAnklePos" value="0.015" />
 	<xacro:property name="legAnklePos" value="0" />
-	<xacro:property name="lowerKneePos" value="0.0.12" />
+	<xacro:property name="lowerKneePos" value="0.12" />
 	<xacro:property name="upperKneePos" value="0.02" />
-	<xacro:property name="legHipPos" value="0.0132" />
-	<xacro:property name="bodyHipHigth" value="0.01" />
-	<xacro:property name="bodyHipDepth" value="0.025" />
+	<xacro:property name="legHipPos" value="0.132" />
+	<xacro:property name="bodyHipHeight" value="0.01" />
+	<xacro:property name="bodyHipWidth" value="0.025" />
 	<xacro:property name="massJointBodyDepth" value="0.07" />
 	<xacro:property name="massJointBodyHeight" value="0.055" />
@@ -46,15 +46,9 @@
 	<xacro:include filename="$(find dacbot_description)/urdf/dacbot.gazebo" />
 	<xacro:include filename="$(find dacbot_description)/urdf/colors.xacro" />
-	<!-- Used for fixing robot to Gazebo 'base_link' -->
-	<link name="world"/>
-	<joint name="fixed_left" type="fixed">
-		<parent link="world"/>
-		<child link="left_foot"/>
-	</joint>
 	<!--
 		Macros
 	 -->
 	 <!-- Box Macro!
-	<xacro:box name="" origin_x="" origin_y="" origin_z="" width="" length="" height="" mass="" />
+	<xacro:create_box name="" origin_x="" origin_y="" origin_z="" width="" length="" height="" mass="" />
 	 -->
 	<xacro:macro name="create_box" params="name origin_x origin_y origin_z width length height mass">
@@ -87,38 +81,76 @@
 	-->
 	<!-- Left Foot -->
-	<xacro:property name="var" value="1"/>
-	<xacro:create_box name="left_foot" origin_x="${var}" origin_y="${footLength*scale/2 - footAnklePos}" origin_z="${footHeight/2}" width="${footWidth}" length="${footLength}" height="${footHeight}" mass="${footMass}" />
-	<!-- Left Foot -->
-	<xacro:property name="var" value"${var} + 1"/>
-	<xacro:create_box name="left_lower_leg" origin_x="${var}" origin_y="${footLength*scale/2 - footAnklePos}" origin_z="${footHeight/2}" width="${footWidth}" length="${footLength}" height="${footHeight}" mass="${footMass}" />
+	<xacro:create_box name="left_foot" origin_x="${-legDistFromCenter}" origin_y="${footLength*scale/2 - footAnklePos}" origin_z="${footHeight/2}" width="${footWidth}" length="${footLength}" height="${footHeight}" mass="${footMass}" />
 	<!-- Left Lower Leg -->
+	<xacro:create_box name="left_lower_leg" origin_x="${-legDistFromCenter}" origin_y="0" origin_z="${lowerLegHeight/2 + footHeight - legAnklePos}" width="${lowerLegWidth}" length="${lowerLegLength}" height="${lowerLegHeight}" mass="${lowerLegMass}" />
+	<!-- Left Upper Leg -->
+	<xacro:create_box name="left_upper_leg" origin_x="${-legDistFromCenter}" origin_y="0" origin_z="${upperLegHeight/2 + footHeight - legAnklePos + lowerKneePos - upperKneePos}" width="${upperLegWidth}" length="${upperLegLength}" height="${upperLegHeight}" mass="${upperLegMass}" />
 	<!--
-	<link name="left_lower_leg">
-		<collision>
-			<origin xyz="${-legDistFromCenter} 0 ${footHeight + lowerLegHeight*scale/2}" rpy="0 0 0"/>
-			<geometry>
-				<box size="${lowerLegWidth*scale} ${lowerLegLength*scale} ${lowerLegHeight*scale}" />
-			</geometry>
-		</collision>
-		<visual>
-			<origin xyz="${-bodyWidth/2} 0 ${footHeight + lowerLegHeight/2}" rpy="0 0 0"/>
-			<geometry>
-				<box size="${lowerLegWidth*scale} ${lowerLegLength*scale} ${lowerLegHeight*scale}" />
-			</geometry>
-			<material name="orange"/>
-		</visual>
-		<inertial>
-			<origin xyz="${-bodyWidth/2} 0 ${footHeight + lowerLegHeight/2}" rpy="0 0 0"/>
-			<mass value="${footMass}"/>
-			<inertia
-				ixx="${footMass / 12.0 * (lowerLegWidth*lowerLegWidth + lowerLegHeight*lowerLegHeight)}" ixy="0.0" ixz="0.0"
-				iyy="${footMass / 12.0 * (lowerLegHeight*lowerLegHeight + lowerLegWidth*lowerLegWidth)}" iyz="0.0"
-				izz="${footMass / 12.0 * (lowerLegWidth*lowerLegWidth + lowerLegWidth*lowerLegWidth)}"/>
-		</inertial>
-	</link>
-	<joint name="left_ankle" type="fixed">
+		Right Leg
+	-->
+	<!-- Right Foot -->
+	<xacro:create_box name="right_foot" origin_x="${legDistFromCenter}" origin_y="${footLength*scale/2 - footAnklePos}" origin_z="${footHeight/2}" width="${footWidth}" length="${footLength}" height="${footHeight}" mass="${footMass}" />
+	<!-- Right Lower Leg -->
+	<xacro:create_box name="right_lower_leg" origin_x="${legDistFromCenter}" origin_y="0" origin_z="${lowerLegHeight/2 + footHeight - legAnklePos}" width="${lowerLegWidth}" length="${lowerLegLength}" height="${lowerLegHeight}" mass="${lowerLegMass}" />
+	<!-- Right Upper Leg -->
+	<xacro:create_box name="right_upper_leg" origin_x="${legDistFromCenter}" origin_y="0" origin_z="${upperLegHeight/2 + footHeight - legAnklePos + lowerKneePos - upperKneePos}" width="${upperLegWidth}" length="${upperLegLength}" height="${upperLegHeight}" mass="${upperLegMass}" />
+	<!--
+		Body
+	-->
+	<xacro:create_box name="body" origin_x="0" origin_y="${bodyWidth/2 - bodyHipWidth}" origin_z="${bodyHeight/2 + footHeight - legAnklePos + lowerKneePos - upperKneePos + legHipPos - bodyHipHeight}" width="${bodyWidth}" length="${bodyLength}" height="${bodyHeight}" mass="${bodyMass}" />
+	<!--
+		Joints
+	-->
+	<!-- Used for fixing robot to Gazebo 'base_link' -->
+	<link name="world"/>
+	<joint name="world_left_foot" type="floating">
+		<parent link="world"/>
+		<child link="left_foot"/>
+	</joint>
+	<joint name="world_right_foot" type="floating">
+		<parent link="world"/>
+		<child link="right_foot"/>
+	</joint>
+	<joint name="left_ankle" type="continuous">
 		<parent link="left_foot"/>
 		<child link="left_lower_leg"/>
+		<origin xyz="${-legDistFromCenter} 0 ${footHeight/2}" rpy="0 0 0"/>
+		<axis xyz="1 0 0"/>
+		<dynamics damping="0.7"/>
 	</joint>
--->
+	<joint name="left_knee" type="fixed">
+		<parent link="left_lower_leg"/>
+		<child link="left_upper_leg"/>
+		<origin xyz="${-legDistFromCenter} 0 0" rpy="0 0 0"/>
+		<axis xyz="1 0 0"/>
+		<dynamics damping="0.7"/>
+	</joint>
+	<joint name="left_hip" type="continuous">
+		<parent link="left_upper_leg"/>
+		<child link="body"/>
+		<origin xyz="${-legDistFromCenter} 0 0" rpy="0 0 0"/>
+		<axis xyz="1 0 0"/>
+		<dynamics damping="0.7"/>
+	</joint>
+	<joint name="right_ankle" type="continuous">
+		<parent link="right_foot"/>
+		<child link="right_lower_leg"/>
+		<origin xyz="${-legDistFromCenter} 0 ${footHeight/2}" rpy="0 0 0"/>
+		<axis xyz="1 0 0"/>
+		<dynamics damping="0.7"/>
+	</joint>
+	<joint name="right_knee" type="fixed">
+		<parent link="right_lower_leg"/>
+		<child link="right_upper_leg"/>
+		<origin xyz="${-legDistFromCenter} 0 0" rpy="0 0 0"/>
+		<axis xyz="1 0 0"/>
+		<dynamics damping="0.7"/>
+	</joint>
+	<joint name="right_hip" type="continuous">
+		<parent link="right_upper_leg"/>
+		<child link="body"/>
+		<origin xyz="${-legDistFromCenter} 0 0" rpy="0 0 0"/>
+		<axis xyz="1 0 0"/>
+		<dynamics damping="0.7"/>
+	</joint>
 </robot>

Commit message: all parts added and compiles, but doesnt work yet!

File: src/dacbot_description/urdf/dacbot.xacro (robot description, xacro)
@@ -154,3 +154,26 @@
 		<dynamics damping="0.7"/>
 	</joint>
+	<!--
+		Transmissions
+	-->
+	<transmission name="transmission_left_knee">
+		<type>transmission_interface/SimpleTransmission</type>
+		<joint name="left_knee">
+			<hardwareInterface>EffortJointInterface</hardwareInterface>
+		</joint>
+		<actuator name="motor_left_knee">
+			<hardwareInterface>EffortJointInterface</hardwareInterface>
+			<mechanicalReduction>1</mechanicalReduction>
+		</actuator>
+	</transmission>
+	<transmission name="transmission_left_hip">
+		<type>transmission_interface/SimpleTransmission</type>
+		<joint name="left_hip">
+			<hardwareInterface>EffortJointInterface</hardwareInterface>
+		</joint>
+		<actuator name="motor_left_hip">
+			<hardwareInterface>EffortJointInterface</hardwareInterface>
+			<mechanicalReduction>1</mechanicalReduction>
+		</actuator>
+	</transmission>
 </robot>

Commit message: it moves! the joint are wrong but it moves!

File: src/dacbot_description/urdf/dacbot.xacro (robot description, xacro)
@@ -154,26 +154,3 @@
 		<dynamics damping="0.7"/>
 	</joint>
-	<!--
-		Transmissions
-	-->
-	<transmission name="transmission_left_knee">
-		<type>transmission_interface/SimpleTransmission</type>
-		<joint name="left_knee">
-			<hardwareInterface>EffortJointInterface</hardwareInterface>
-		</joint>
-		<actuator name="motor_left_knee">
-			<hardwareInterface>EffortJointInterface</hardwareInterface>
-			<mechanicalReduction>1</mechanicalReduction>
-		</actuator>
-	</transmission>
-	<transmission name="transmission_left_hip">
-		<type>transmission_interface/SimpleTransmission</type>
-		<joint name="left_hip">
-			<hardwareInterface>EffortJointInterface</hardwareInterface>
-		</joint>
-		<actuator name="motor_left_hip">
-			<hardwareInterface>EffortJointInterface</hardwareInterface>
-			<mechanicalReduction>1</mechanicalReduction>
-		</actuator>
-	</transmission>
 </robot>

Commit message: Using another property and reduced minimum intertia to 0.002

File: src/dacbot_description/urdf/dacbot.xacro (robot description, xacro)
@@ -9,4 +9,5 @@
 	-->
 	<xacro:property name="scale" value="1" />
+	<xacro:property name="minimum_intertia" value="0.002" /> <!-- <0.001 doesn't work -->
 	<xacro:property name="bodyWidth" value="${0.085*scale}" />
 	<xacro:property name="bodyLength" value="${0.08*scale}" />
@@ -53,14 +54,14 @@
 	 -->
 	<xacro:macro name="create_box" params="name origin_x origin_y origin_z r p y width length height mass">
-		<!-- Set the minimum intertia as 0.01 -->
-		<xacro:property name="ixx" value="0.01" />
+		<!-- Set the minimum intertia -->
+		<xacro:property name="ixx" value="${minimum_intertia}" />
 		<xacro:if value="${mass / 12.0 * (length*length + height*height) > 0.01}">
 			<xacro:property name="ixx" value="${mass / 12.0 * (length*length + height*height)}" />
 		</xacro:if>
-		<xacro:property name="iyy" value="0.01" />
+		<xacro:property name="iyy" value="${minimum_intertia}" />
 		<xacro:if value="${mass / 12.0 * (length*length + height*height) > 0.01}">
 			<xacro:property name="iyy" value="${mass / 12.0 * (length*length + height*height)}" />
 		</xacro:if>
-		<xacro:property name="izz" value="0.01" />
+		<xacro:property name="izz" value="${minimum_intertia}" />
 		<xacro:if value="${mass / 12.0 * (length*length + height*height) > 0.01}">
 			<xacro:property name="izz" value="${mass / 12.0 * (length*length + height*height)}" />

Commit message: Added virtual transmission for mapping the output from the controller to the actuator

File: src/dacbot_description/urdf/dacbot.xacro (robot description, xacro)
@@ -3,5 +3,7 @@
 	<!-- Constants -->
 	<xacro:property name="PI" value="3.1415926535897931"/>
-	<!-- Robot configuration
+	<!-- Robot configuration: Transmission -->
+	<xacro:property name="maxRealMotorTorque" value="1.0787315"/> <!-- In N*m -->
+	<!-- Robot configuration: Geometry
 		Width = X axis
 		Length = Y axis
@@ -176,5 +178,5 @@
 		<actuator name="left_hip_motor">
 			<hardwareInterface>EffortJointInterface</hardwareInterface>
-			<mechanicalReduction>1</mechanicalReduction>
+			<mechanicalReduction>${maxRealMotorTorque}</mechanicalReduction>
 		</actuator>
 	</transmission>
@@ -186,5 +188,5 @@
 		<actuator name="left_knee_motor">
 			<hardwareInterface>EffortJointInterface</hardwareInterface>
-			<mechanicalReduction>1</mechanicalReduction>
+			<mechanicalReduction>${maxRealMotorTorque}</mechanicalReduction>
 		</actuator>
 	</transmission>
@@ -196,5 +198,5 @@
 		<actuator name="left_ankle_motor">
 			<hardwareInterface>EffortJointInterface</hardwareInterface>
-			<mechanicalReduction>1</mechanicalReduction>
+			<mechanicalReduction>${maxRealMotorTorque}</mechanicalReduction>
 		</actuator>
 	</transmission>
@@ -206,5 +208,5 @@
 		<actuator name="right_hip_motor">
 			<hardwareInterface>EffortJointInterface</hardwareInterface>
-			<mechanicalReduction>1</mechanicalReduction>
+			<mechanicalReduction>${maxRealMotorTorque}</mechanicalReduction>
 		</actuator>
 	</transmission>
@@ -216,5 +218,5 @@
 		<actuator name="right_knee_motor">
 			<hardwareInterface>EffortJointInterface</hardwareInterface>
-			<mechanicalReduction>1</mechanicalReduction>
+			<mechanicalReduction>${maxRealMotorTorque}</mechanicalReduction>
 		</actuator>
 	</transmission>
@@ -226,5 +228,5 @@
 		<actuator name="right_ankle_motor">
 			<hardwareInterface>EffortJointInterface</hardwareInterface>
-			<mechanicalReduction>1</mechanicalReduction>
+			<mechanicalReduction>${maxRealMotorTorque}</mechanicalReduction>
 		</actuator>
 	</transmission>

Commit message: Added limits to the joints

File: src/dacbot_description/urdf/dacbot.xacro (robot description, xacro)
@@ -3,9 +3,10 @@
 	<!-- Constants -->
 	<xacro:property name="PI" value="3.1415926535897931"/>
+	<xacro:property name="DEG_TO_RAD" value="${PI/180}"/>
 	<!-- ROS -->
 	<xacro:property name="update_rate" value="2"/>
 	<xacro:property name="robot_name" value="dacbot"/>
 	<!-- Robot configuration: Transmission -->
-	<xacro:property name="maxRealMotorTorque" value="1.0787315"/> <!-- In N*m -->
+	<xacro:property name="maxRealMotorTorque" value="2.0787315"/> <!-- In N*m -->
 	<!-- Robot configuration: Geometry
 		Width = X axis
@@ -132,45 +133,51 @@
     <origin xyz="0 0 ${(footHeight + lowerLegHeight + upperLegHeight)*1.1}" rpy="0 0 0"/>
   </joint>  -->
-	<joint name="left_hip" type="continuous">
+	<joint name="left_hip" type="revolute">
 		<parent link="body"/>
 		<child link="left_upper_leg"/>
 		<origin xyz="${-legDistFromCenter} 0 0" rpy="0 ${PI/2} 0"/>
 		<axis xyz="0 0 1"/>
-		<dynamics damping="0.7"/>
-	</joint>
-	<joint name="left_knee" type="continuous">
+		<limit effort="10" velocity="1.0" lower="-${78*DEG_TO_RAD}" upper="${100*DEG_TO_RAD}" />
+		<dynamics damping="0.7"/>
+	</joint>
+	<joint name="left_knee" type="revolute">
 		<parent link="left_upper_leg"/>
 		<child link="left_lower_leg"/>
 		<origin xyz="${upperLegHeight} 0 0" rpy="0 0 0"/>
 		<axis xyz="0 0 1"/>
-		<dynamics damping="0.7"/>
-	</joint>
-	<joint name="left_ankle" type="continuous">
+		<limit effort="10" velocity="1.0" lower="-${150*DEG_TO_RAD}" upper="0" />
+		<dynamics damping="0.7"/>
+	</joint>
+	<joint name="left_ankle" type="revolute">
 		<parent link="left_lower_leg"/>
 		<child link="left_foot"/>
 		<origin xyz="${lowerLegHeight} 0 0" rpy="0 0 0"/>
 		<axis xyz="0 0 1"/>
-		<dynamics damping="0.7"/>
-	</joint>
-	<joint name="right_hip" type="continuous">
+		<!-- <limit effort="10" velocity="1.0" lower="-${90*DEG_TO_RAD}" upper="${30*DEG_TO_RAD}" /> -->
+		<limit effort="10" velocity="1.0" lower="0" upper="0" />
+		<dynamics damping="0.7"/>
+	</joint>
+	<joint name="right_hip" type="revolute">
 		<parent link="body"/>
 		<child link="right_upper_leg"/>
 		<origin xyz="${legDistFromCenter} 0 0" rpy="0 ${PI/2} 0"/>
 		<axis xyz="0 0 1"/>
-		<dynamics damping="0.7"/>
-	</joint>
-	<joint name="right_knee" type="continuous">
+		<limit effort="10" velocity="1.0" lower="-${78*DEG_TO_RAD}" upper="${100*DEG_TO_RAD}" />
+	</joint>
+	<joint name="right_knee" type="revolute">
 		<parent link="right_upper_leg"/>
 		<child link="right_lower_leg"/>
 		<origin xyz="${upperLegHeight} 0 0" rpy="0 0 0"/>
 		<axis xyz="0 0 1"/>
-		<dynamics damping="0.7"/>
-	</joint>
-	<joint name="right_ankle" type="continuous">
+		<limit effort="10" velocity="1.0" lower="-${150*DEG_TO_RAD}" upper="0" />
+		<dynamics damping="0.7"/>
+	</joint>
+	<joint name="right_ankle" type="revolute">
 		<parent link="right_lower_leg"/>
 		<child link="right_foot"/>
 		<origin xyz="${lowerLegHeight} 0 0" rpy="0 0 0"/>
 		<axis xyz="0 0 1"/>
-		<dynamics damping="0.7"/>
+		<!-- <limit effort="10" velocity="1.0" lower="-${90*DEG_TO_RAD}" upper="${30*DEG_TO_RAD}" /> -->
+		<limit effort="10" velocity="1.0" lower="0" upper="0" />
 	</joint>
 	<transmission name="left_hip_trans">

Commit message: Spedded up

File: src/dacbot_description/urdf/dacbot.xacro (robot description, xacro)
@@ -8,5 +8,5 @@
 	<xacro:property name="robot_name" value="dacbot"/>
 	<!-- Robot configuration: Transmission -->
-	<xacro:property name="maxRealMotorTorque" value="2.0787315"/> <!-- In N*m -->
+	<xacro:property name="maxRealMotorTorque" value="1.0787315"/> <!-- In N*m -->
 	<!-- Robot configuration: Geometry
 		Width = X axis
