Commit message: The description of the rotational platform is now inside of the robot description so we can use the flag "robot floating" to debug the gaits

File: src/dacbot_description/urdf/dacbot.xacro (robot description, xacro)
@@ -5,8 +5,9 @@
 	<xacro:property name="DEG_TO_RAD" value="${PI/180}"/>
 	<!-- ROS -->
-	<xacro:property name="update_rate" value="2"/>
+	<xacro:property name="update_rate" value="10"/>
 	<xacro:property name="robot_name" value="dacbot"/>
 	<!-- Robot configuration: Transmission -->
-	<xacro:property name="maxRealMotorTorque" value="1.0787315"/> <!-- In N*m -->
+	<xacro:property name="max_real_motor_torque" value="1.0787315"/> <!-- In N*m -->
+  <xacro:property name="robot_floating" value="1"/>
 	<!-- Robot configuration: Geometry
 		Width = X axis
@@ -188,5 +189,5 @@
 		<actuator name="left_hip_motor">
 			<hardwareInterface>EffortJointInterface</hardwareInterface>
-			<mechanicalReduction>${maxRealMotorTorque}</mechanicalReduction>
+			<mechanicalReduction>${max_real_motor_torque}</mechanicalReduction>
 		</actuator>
 	</transmission>
@@ -198,5 +199,5 @@
 		<actuator name="left_knee_motor">
 			<hardwareInterface>EffortJointInterface</hardwareInterface>
-			<mechanicalReduction>${maxRealMotorTorque}</mechanicalReduction>
+			<mechanicalReduction>${max_real_motor_torque}</mechanicalReduction>
 		</actuator>
 	</transmission>
@@ -208,5 +209,5 @@
 		<actuator name="left_ankle_motor">
 			<hardwareInterface>EffortJointInterface</hardwareInterface>
-			<mechanicalReduction>${maxRealMotorTorque}</mechanicalReduction>
+			<mechanicalReduction>${max_real_motor_torque}</mechanicalReduction>
 		</actuator>
 	</transmission>
@@ -218,5 +219,5 @@
 		<actuator name="right_hip_motor">
 			<hardwareInterface>EffortJointInterface</hardwareInterface>
-			<mechanicalReduction>${maxRealMotorTorque}</mechanicalReduction>
+			<mechanicalReduction>${max_real_motor_torque}</mechanicalReduction>
 		</actuator>
 	</transmission>
@@ -228,5 +229,5 @@
 		<actuator name="right_knee_motor">
 			<hardwareInterface>EffortJointInterface</hardwareInterface>
-			<mechanicalReduction>${maxRealMotorTorque}</mechanicalReduction>
+			<mechanicalReduction>${max_real_motor_torque}</mechanicalReduction>
 		</actuator>
 	</transmission>
@@ -238,12 +239,113 @@
 		<actuator name="right_ankle_motor">
 			<hardwareInterface>EffortJointInterface</hardwareInterface>
-			<mechanicalReduction>${maxRealMotorTorque}</mechanicalReduction>
+			<mechanicalReduction>${max_real_motor_torque}</mechanicalReduction>
 		</actuator>
 	</transmission>
 	<!-- Rotational robot holder -->
-	<xacro:property name="rotational_robot_holder_base_radius" value="${0.2*scale}" />
-  <xacro:property name="rotational_robot_holder_base_length" value="${(footHeight + lowerLegHeight + upperLegHeight)*scale}" />
+  <xacro:property name="rotational_robot_holder_base_length_extra" value="0" />
+  <xacro:if value="${robot_floating is 1}">
+    <xacro:property name="rotational_robot_holder_base_length_extra" value="0.1" />
+  </xacro:if>
+  <xacro:property name="rotational_robot_holder_base_length" value="${(footHeight + lowerLegHeight + upperLegHeight + rotational_robot_holder_base_length_extra)*scale}" />
+  <xacro:property name="rotational_robot_holder_base_radius" value="${0.2*scale}" />
   <xacro:property name="rotational_robot_holder_holder_radius" value="${0.01*scale}" />
   <xacro:property name="rotational_robot_holder_holder_length" value="${2*scale}" />
-	<xacro:include filename="$(find gazebo_resources)/models/rotational_robot_holder/urdf/rotational_robot_holder.xacro" />
+	<!-- <xacro:include filename="$(find gazebo_resources)/models/rotational_robot_holder/urdf/rotational_robot_holder.xacro" /> -->
+  <link name="rotational_robot_holder_base">
+    <collision>
+      <origin xyz="0 0 0" rpy="0 0 0"/>
+      <geometry>
+        <cylinder length="${rotational_robot_holder_base_length}" radius="${rotational_robot_holder_base_radius}"/>
+      </geometry>
+    </collision>
+    <visual>
+      <origin xyz="0 0 0" rpy="0 0 0"/>
+      <geometry>
+        <cylinder length="${rotational_robot_holder_base_length}" radius="${rotational_robot_holder_base_radius}"/>
+      </geometry>
+      <material name="orange"/>
+    </visual>
+    <inertial>
+      <mass value="10"/>
+      <inertia ixx="0.4" ixy="0.0" ixz="0.0" iyy="0.4" iyz="0.0" izz="0.2"/>
+    </inertial>
+  </link>
+  <link name="rotational_robot_holder_virtual">
+    <collision>
+      <origin xyz="0 0 0" rpy="0 0 0"/>
+      <geometry>
+        <sphere radius="0.01"/>
+      </geometry>
+    </collision>
+    <visual>
+      <origin xyz="0 0 0" rpy="0 0 0"/>
+      <geometry>
+         <sphere radius="0.01"/>
+      </geometry>
+      <material name="orange"/>
+    </visual>
+    <inertial>
+      <mass value="0.01"/>
+      <inertia ixx="0.1" ixy="0.0" ixz="0.0" iyy="0.1" iyz="0.0" izz="0.1"/>
+    </inertial>
+  </link>
+  <link name="rotational_robot_holder_holder">
+    <collision>
+      <origin xyz="${rotational_robot_holder_holder_length/2} 0 0" rpy="0 ${PI/2} 0"/>
+      <geometry>
+        <cylinder length="${rotational_robot_holder_holder_length}" radius="${rotational_robot_holder_holder_radius}"/>
+      </geometry>
+    </collision>
+    <visual>
+      <origin xyz="${rotational_robot_holder_holder_length/2} 0 0" rpy="0 ${PI/2} 0"/>
+      <geometry>
+         <cylinder length="${rotational_robot_holder_holder_length}" radius="${rotational_robot_holder_holder_radius}"/>
+      </geometry>
+      <material name="orange"/>
+    </visual>
+    <inertial>
+      <mass value="0.01"/>
+      <inertia ixx="0.1" ixy="0.0" ixz="0.0" iyy="0.1" iyz="0.0" izz="0.1"/>
+    </inertial>
+  </link>
+  <!-- Robot to rotational_robot_holder -->
+  <joint name="rotational_robot_holder_base_to_world" type="fixed">
+    <parent link="world"/>
+    <child link="rotational_robot_holder_base"/>
+    <origin xyz="0 0 ${rotational_robot_holder_base_length/2}" rpy="0 0 0"/>
+  </joint>
+  <xacro:if value="${robot_floating is 1}">
+    <joint name="rotational_robot_holder_virtual_to_holder" type="fixed">
+      <parent link="rotational_robot_holder_base"/>
+      <child link="rotational_robot_holder_virtual"/>
+    </joint>
+    <joint name="rotational_robot_holder_joint" type="fixed">
+      <parent link="rotational_robot_holder_virtual"/>
+      <child link="rotational_robot_holder_holder"/>
+      <origin xyz="0 0 ${rotational_robot_holder_base_length/2}" rpy="0 0 0"/>
+    </joint>
+  </xacro:if>
+  <xacro:if value="${robot_floating is 0}">
+    <joint name="rotational_robot_holder_virtual_to_holder" type="continuous">
+      <parent link="rotational_robot_holder_base"/>
+      <child link="rotational_robot_holder_virtual"/>
+      <origin xyz="0 0 0" rpy="0 0 0"/>
+      <axis xyz="0 1 0"/>
+      <dynamics damping="0.7"/>
+    </joint>
+    <joint name="rotational_robot_holder_joint" type="continuous">
+      <parent link="rotational_robot_holder_virtual"/>
+      <child link="rotational_robot_holder_holder"/>
+      <origin xyz="0 0 ${rotational_robot_holder_base_length/2}" rpy="0 0 0"/>
+      <axis xyz="0 0 1"/>
+      <dynamics damping="0.7"/>
+    </joint>
+  </xacro:if>
+  <joint name="rotational_robot_holder_to_rotot" type="fixed">
+    <parent link="rotational_robot_holder_holder"/>
+    <child link="body"/>
+    <origin xyz="${rotational_robot_holder_holder_length+bodyWidth/2} 0 0" rpy="0 0 0"/>
+    <axis xyz="0 0 1"/>
+    <limit effort="30" velocity="1.0" lower="0" upper="1" />
+  </joint>
 </robot>

Commit message: joints limits and damping parameters as xacro properties

File: src/dacbot_description/urdf/dacbot.xacro (robot description, xacro)
@@ -7,14 +7,16 @@
 	<xacro:property name="update_rate" value="10"/>
 	<xacro:property name="robot_name" value="dacbot"/>
+  <!-- Robot configuration: Miscellaneous -->
+  <xacro:property name="robot_floating" value="0"/>
 	<!-- Robot configuration: Transmission -->
 	<xacro:property name="max_real_motor_torque" value="1.0787315"/> <!-- In N*m -->
-  <xacro:property name="robot_floating" value="1"/>
-	<!-- Robot configuration: Geometry
-		Width = X axis
-		Length = Y axis
-		Height = Z axis
-	-->
-	<xacro:property name="scale" value="1" />
-	<xacro:property name="minimum_intertia" value="0.002" /> <!-- <0.001 doesn't work -->
+  <!-- Robot configuration: Geometry
+    Width = X axis
+    Length = Y axis
+    Height = Z axis
+  -->
+  <xacro:property name="scale" value="1" />
+  <xacro:property name="minimum_intertia" value="0.002" /> <!-- <0.001 doesn't work -->
+  <xacro:property name="damping" value="0.8"/>
 	<xacro:property name="bodyWidth" value="${0.085*scale}" />
 	<xacro:property name="bodyLength" value="${0.08*scale}" />
@@ -29,12 +31,27 @@
 	<xacro:property name="upperLegHeight" value="${0.142*scale}" />
 	<xacro:property name="upperLegMass" value="${0.2*scale}" />
+  <xacro:property name="upperLegLimitUpperPosition" value="70" />
+  <xacro:property name="upperLegLimitLowerPosition" value="-70" />
+  <xacro:property name="upperLegLimitVelocity" value="10" />
+  <xacro:property name="upperLegLimitEffort" value="10" />
+  <xacro:property name="upperLegDamping" value="0.7" />
 	<xacro:property name="lowerLegWidth" value="${0.015*scale}" />
 	<xacro:property name="lowerLegLength" value="${0.015*scale}" />
 	<xacro:property name="lowerLegHeight" value="${0.125*scale}" />
 	<xacro:property name="lowerLegMass" value="${0.08*scale}" />
+  <xacro:property name="lowerLegLimitUpperPosition" value="0" />
+  <xacro:property name="lowerLegLimitLowerPosition" value="150" />
+  <xacro:property name="lowerLegLimitVelocity" value="10" />
+  <xacro:property name="lowerLegLimitEffort" value="10" />
+  <xacro:property name="lowerLegDamping" value="0.7" />
 	<xacro:property name="footWidth" value="${0.015*scale}" />
 	<xacro:property name="footLength" value="${0.050*scale}" />
 	<xacro:property name="footHeight" value="${0.008*scale}" />
 	<xacro:property name="footMass" value="${0.01*scale}" />
+  <xacro:property name="footLimitUpperPosition" value="0" />
+  <xacro:property name="footLimitLowerPosition" value="0" />
+  <xacro:property name="footLimitVelocity" value="10" />
+  <xacro:property name="footLimitEffort" value="10" />
+  <xacro:property name="footDamping" value="0.7" />
 	<xacro:property name="legDistFromCenter" value="${0.015*scale}" />
 	<xacro:property name="footAnklePos" value="${0.015*scale}" />
@@ -139,6 +156,6 @@
 		<origin xyz="${-legDistFromCenter} 0 0" rpy="0 ${PI/2} 0"/>
 		<axis xyz="0 0 1"/>
-		<limit effort="10" velocity="1.0" lower="-${78*DEG_TO_RAD}" upper="${100*DEG_TO_RAD}" />
-		<dynamics damping="0.7"/>
+		<limit effort="${upperLegLimitEffort}" velocity="${upperLegLimitVelocity}" lower="${upperLegLimitLowerPosition*DEG_TO_RAD}" upper="${upperLegLimitUpperPosition*DEG_TO_RAD}" />
+		<dynamics damping="${upperLegDamping}"/>
 	</joint>
 	<joint name="left_knee" type="revolute">
@@ -147,6 +164,6 @@
 		<origin xyz="${upperLegHeight} 0 0" rpy="0 0 0"/>
 		<axis xyz="0 0 1"/>
-		<limit effort="10" velocity="1.0" lower="-${150*DEG_TO_RAD}" upper="0" />
-		<dynamics damping="0.7"/>
+		<limit effort="${lowerLegLimitEffort}" velocity="${lowerLegLimitVelocity}" lower="${lowerLegLimitLowerPosition*DEG_TO_RAD}" upper="${lowerLegLimitUpperPosition*DEG_TO_RAD}" />
+		<dynamics damping="${lowerLegDamping}"/>
 	</joint>
 	<joint name="left_ankle" type="revolute">
@@ -155,7 +172,6 @@
 		<origin xyz="${lowerLegHeight} 0 0" rpy="0 0 0"/>
 		<axis xyz="0 0 1"/>
-		<!-- <limit effort="10" velocity="1.0" lower="-${90*DEG_TO_RAD}" upper="${30*DEG_TO_RAD}" /> -->
-		<limit effort="10" velocity="1.0" lower="0" upper="0" />
-		<dynamics damping="0.7"/>
+		<limit effort="${footLimitEffort}" velocity="${footLimitVelocity}" lower="${footLimitLowerPosition}" upper="${footLimitUpperPosition}" />
+		<dynamics damping="${footDamping}"/>
 	</joint>
 	<joint name="right_hip" type="revolute">
@@ -164,5 +180,6 @@
 		<origin xyz="${legDistFromCenter} 0 0" rpy="0 ${PI/2} 0"/>
 		<axis xyz="0 0 1"/>
-		<limit effort="10" velocity="1.0" lower="-${78*DEG_TO_RAD}" upper="${100*DEG_TO_RAD}" />
+    <limit effort="${upperLegLimitEffort}" velocity="${upperLegLimitVelocity}" lower="${upperLegLimitLowerPosition*DEG_TO_RAD}" upper="${upperLegLimitUpperPosition*DEG_TO_RAD}" />
+    <dynamics damping="${upperLegDamping}"/>
 	</joint>
 	<joint name="right_knee" type="revolute">
@@ -171,6 +188,6 @@
 		<origin xyz="${upperLegHeight} 0 0" rpy="0 0 0"/>
 		<axis xyz="0 0 1"/>
-		<limit effort="10" velocity="1.0" lower="-${150*DEG_TO_RAD}" upper="0" />
-		<dynamics damping="0.7"/>
+    <limit effort="${lowerLegLimitEffort}" velocity="${lowerLegLimitVelocity}" lower="${lowerLegLimitLowerPosition*DEG_TO_RAD}" upper="${lowerLegLimitUpperPosition*DEG_TO_RAD}" />
+		<dynamics damping="${lowerLegDamping}"/>
 	</joint>
 	<joint name="right_ankle" type="revolute">
@@ -179,6 +196,6 @@
 		<origin xyz="${lowerLegHeight} 0 0" rpy="0 0 0"/>
 		<axis xyz="0 0 1"/>
-		<!-- <limit effort="10" velocity="1.0" lower="-${90*DEG_TO_RAD}" upper="${30*DEG_TO_RAD}" /> -->
-		<limit effort="10" velocity="1.0" lower="0" upper="0" />
+		<limit effort="${footLimitEffort}" velocity="${footLimitVelocity}" lower="${footLimitLowerPosition}" upper="${footLimitUpperPosition}" />
+    <dynamics damping="${footDamping}"/>
 	</joint>
 	<transmission name="left_hip_trans">

Commit message: fixed bug when scaling the rotational holder

File: src/dacbot_description/urdf/dacbot.xacro (robot description, xacro)
@@ -17,5 +17,5 @@
   -->
   <xacro:property name="scale" value="1" />
-  <xacro:property name="minimum_intertia" value="0.002" /> <!-- <0.001 doesn't work -->
+  <xacro:property name="minimum_intertia" value="2e-03" /> <!-- <0.001 doesn't work -->
 	<xacro:property name="bodyWidth" value="${0.085*scale}" />
 	<xacro:property name="bodyLength" value="${0.08*scale}" />
@@ -263,5 +263,5 @@
     <xacro:property name="rotational_robot_holder_base_length_extra" value="0.1" />
   </xacro:if>
-  <xacro:property name="rotational_robot_holder_base_length" value="${(footHeight + lowerLegHeight + upperLegHeight + rotational_robot_holder_base_length_extra)*scale}" />
+  <xacro:property name="rotational_robot_holder_base_length" value="${(footHeight + lowerLegHeight + upperLegHeight + rotational_robot_holder_base_length_extra)}" />
   <xacro:property name="rotational_robot_holder_base_radius" value="${0.2*scale}" />
   <xacro:property name="rotational_robot_holder_holder_radius" value="${0.01*scale}" />
