Commit message: floating

File: src/legs_description/urdf/legs_false_inertias.xacro (robot description, xacro)
@@ -218,11 +218,11 @@
     <child link="hip"/>
     <axis xyz="0 1 0"/>
-  </joint>
-  -->
-  <joint name="world_hip" type="floating">
+  </joint> -->
+<!--
+  <joint name="world_hip" type="continuous">
     <origin xyz="0 0 1" rpy="0 0 0"/>
     <parent link="world"/>
     <child link="hip"/>
-  </joint>
+  </joint>  -->
 	<!--
 		Joints
@@ -336,5 +336,5 @@
     </actuator>
   </transmission>
-<!--
+  <!-- Rotational robot holder -->
   <xacro:property name="rotational_robot_holder_base_length_extra" value="0" />
   <xacro:if value="${robot_floating is 1}">
