Commit message: Commit with real inertias. Stack gazebo doesnt work with such small intertias. Thus, either we compile gazebo with other physic simulator or we increase the inertias. Both will be tried.

File: src/legs_description/urdf/legs.urdf (robot description, URDF)
Before this commit: robot legs, 9 links, 8 joints
Links:
- removed link body
- removed link left_lower_leg
- removed link left_upper_leg
- removed link plane_x
- removed link right_lower_leg
- removed link right_upper_leg
- added link hip, mass 0.156; collision cylinder length=0.180 radius=0.025; visual mesh filename=package://legs_description/meshes/iteration_1/gazebo/hip_vi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
- added link left_lower_limb, mass 0.115; collision cylinder length=0.212 radius=0.01; visual mesh filename=package://legs_description/meshes/iteration_1/gazebo/left_l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
- added link left_upper_limb, mass 0.123; collision cylinder length=0.262 radius=0.01; visual mesh filename=package://legs_description/meshes/iteration_1/gazebo/left_u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
- added link right_lower_limb, mass 0.115; collision cylinder length=0.212 radius=0.01; visual mesh filename=package://legs_description/meshes/iteration_1/gazebo/right_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
- added link right_upper_limb, mass 0.123; collision cylinder length=0.262 radius=0.01; visual mesh filename=package://legs_description/meshes/iteration_1/gazebo/right_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
- added link rotational_robot_holder_base, mass 10; collision cylinder length=1 radius=0.2; visual cylinder length=1 radius=0.2
- added link rotational_robot_holder_holder, mass 0.01; collision cylinder length=2 radius=0.01; visual cylinder length=2 radius=0.01
- added link rotational_robot_holder_virtual, mass 0.01; collision sphere radius=0.01; visual sphere radius=0.01
- link left_foot: mass 0.0296 -> 0.021; geometry collision mesh filename=package://legs_description/meshes/iteration_1/gazebo/left_f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; visual mesh filename=package://legs_description/meshes/iteration_1/gazebo/left_f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
- link right_foot: mass 0.0296 -> 0.021; geometry collision mesh filename=package://legs_description/meshes/iteration_1/gazebo/right_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; visual mesh filename=package://legs_description/meshes/iteration_1/gazebo/right_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
Joints:
- removed joint plane_x_body
- removed joint world_plane_x
- added joint rotational_robot_holder_base_to_world: type fixed, parent world, child rotational_robot_holder_base, origin xyz=0 0 0.5 rpy=0 0 0
- added joint rotational_robot_holder_joint: type continuous, parent rotational_robot_holder_virtual, child rotational_robot_holder_holder, origin xyz=0 0 0.5 rpy=0 0 0, axis 0 0 1
- added joint rotational_robot_holder_to_rotot: type fixed, parent rotational_robot_holder_holder, child hip, origin xyz=2.2 0 0 rpy=0 0 0, axis 0 0 1, limit lower=0 upper=1 effort=30 velocity=1.0
- added joint rotational_robot_holder_virtual_to_holder: type continuous, parent rotational_robot_holder_base, child rotational_robot_holder_virtual, origin xyz=0 0 0 rpy=0 0 0, axis 0 1 0
- joint left_ankle: axis 0 0 1 -> 0 0 -1; limit lower=-0.907571211037 upper=0.663225115758 effort=10 velocity=10 -> lower=-0.872664625997 upper=2.09439510239 effort=10 velocity=10; origin xyz=0.212 0 0 rpy=0 0 0 -> xyz=0 0.212 0 rpy=0 0 0; parent left_lower_leg -> left_lower_limb
- joint left_hip: axis 0 0 1 -> 0 0 -1; child left_upper_leg -> left_upper_limb; limit lower=-1.3962634016 upper=1.3962634016 effort=10 velocity=10 -> lower=-1.0471975512 upper=1.57079632679 effort=10 velocity=10; origin xyz=-0.075 0 0 rpy=0 1.57079632679 0 -> xyz=0 0.0635 -0.028867 rpy=-1.57079632679 0 0; parent body -> hip
- joint left_knee: axis 0 0 1 -> 0 0 -1; child left_lower_leg -> left_lower_limb; limit lower=-2.61799387799 upper=0.0 effort=10 velocity=10 -> lower=-2.09439510239 upper=0.0 effort=10 velocity=10; origin xyz=0.262 0 0 rpy=0 0 0 -> xyz=0 0.262 0 rpy=0 0 0; parent left_upper_leg -> left_upper_limb
- joint right_ankle: axis 0 0 1 -> 0 0 -1; limit lower=-0.907571211037 upper=0.663225115758 effort=10 velocity=10 -> lower=-0.872664625997 upper=2.09439510239 effort=10 velocity=10; origin xyz=0.212 0 0 rpy=0 0 0 -> xyz=0 0.212 0 rpy=0 0 0; parent right_lower_leg -> right_lower_limb
- joint right_hip: axis 0 0 1 -> 0 0 -1; child right_upper_leg -> right_upper_limb; limit lower=-1.3962634016 upper=1.3962634016 effort=10 velocity=10 -> lower=-1.0471975512 upper=1.57079632679 effort=10 velocity=10; origin xyz=0.075 0 0 rpy=0 1.57079632679 0 -> xyz=0 -0.0635 -0.028867 rpy=-1.57079632679 0 0; parent body -> hip
- joint right_knee: axis 0 0 1 -> 0 0 -1; child right_lower_leg -> right_lower_limb; limit lower=-2.61799387799 upper=0.0 effort=10 velocity=10 -> lower=-2.09439510239 upper=0.0 effort=10 velocity=10; origin xyz=0.262 0 0 rpy=0 0 0 -> xyz=0 0.262 0 rpy=0 0 0; parent right_upper_leg -> right_upper_limb

File: src/legs_description/urdf/legs.xacro (robot description, xacro)
@@ -11,135 +11,95 @@
 	<!-- Robot configuration: Transmission -->
 	<xacro:property name="max_real_motor_torque" value="1.0787315"/> <!-- In N*m -->
-  <!-- Robot configuration: Geometry
-    Width = X axis
-    Length = Y axis
-    Height = Z axis
-  -->
-  <xacro:property name="scale" value="1" />
-  <xacro:property name="minimum_intertia" value="0.002" /> <!-- <0.001 doesn't work -->
+  <!-- Robot configuration: Geometry -->
+  <xacro:property name="damping" value="0.7" />
   <xacro:property name="upperLegHeight" value="0.262" />
   <xacro:property name="upperLegDiameter" value="0.02" />
-	<xacro:property name="upperLegMass" value="0.163" />
   <xacro:property name="upperLegLimitUpperPosition" value="90" />
   <xacro:property name="upperLegLimitLowerPosition" value="-60" />
   <xacro:property name="upperLegLimitVelocity" value="10" />
   <xacro:property name="upperLegLimitEffort" value="10" />
-  <xacro:property name="upperLegDamping" value="0.7" />
   <xacro:property name="lowerLegHeight" value="0.212" />
   <xacro:property name="lowerLegDiameter" value="0.02" />
-	<xacro:property name="lowerLegMass" value="0.17" />
   <xacro:property name="lowerLegLimitUpperPosition" value="0" />
   <xacro:property name="lowerLegLimitLowerPosition" value="-120" />
   <xacro:property name="lowerLegLimitVelocity" value="10" />
   <xacro:property name="lowerLegLimitEffort" value="10" />
-  <xacro:property name="lowerLegDamping" value="0.7" />
-	<xacro:property name="footMass" value="0.0296" />
   <xacro:property name="footLimitUpperPosition" value="120" />
   <xacro:property name="footLimitLowerPosition" value="-50" />
   <xacro:property name="footLimitVelocity" value="10" />
   <xacro:property name="footLimitEffort" value="10" />
-  <xacro:property name="footDamping" value="0.7" />
-	<xacro:property name="legDistFromCenter" value="0.0635" />
-  <xacro:property name="hipMass" value="${0.45}" />
-	<xacro:property name="footAnklePos" value="${0.015}" />
-	<xacro:property name="legAnklePos" value="${0}" />
-	<xacro:property name="lowerKneePos" value="${0.12}" />
-	<xacro:property name="upperKneePos" value="${0.02}" />
-	<xacro:property name="legHipPos" value="${0.132}" />
-	<xacro:property name="bodyHipHeight" value="${0.01}" />
-	<xacro:property name="bodyHipWidth" value="${0.025}" />
 	<!-- Import Gazebo customizations and colors-->
 	<xacro:include filename="$(find legs_description)/urdf/legs.gazebo" />
 	<xacro:include filename="$(find legs_description)/urdf/colors.xacro" />
 	<!--
-		Macros
-	 -->
-		<!-- Intertia Macro: Set the minimum intertia -->
-<!--   <xacro:macro name="check_minimum_intertia" params="inertia">
-		<xacro:if value="${inertia < 0.01}">
-			<xacro:property name="inertia" value="${mass / 12.0 * (3*(diameter/2)^2 + height^2)}" />
-		</xacro:if>
-    <xacro:if value="${inertia < 0.01}">
-      <xacro:property name="inertia" value="${mass / 12.0 * (3*(diameter/2)^2 + height^2)}" />
-    </xacro:if>
-    <xacro:if value="${inertia < 0.01}">
-      <xacro:property name="inertia" value="${mass / 12.0 * (3*(diameter/2)^2 + height^2)}" />
-    </xacro:if>
-	</xacro:macro>
- -->
-	<!--
-		World
-	-->
-	<!-- <link name="legs_global"/> -->
-	<!--
 		Left Leg
 	-->
     <link name="hip">
       <collision>
+        <origin xyz="0 0 0" rpy="${90*DEG_TO_RAD} 0 0"/>
+        <geometry>
+          <cylinder length="0.180" radius="0.025"/>
+        </geometry>
+      </collision>
+      <visual>
         <origin xyz="0 0 0" rpy="0 0 0"/>
         <geometry>
           <mesh filename="package://legs_description/meshes/iteration_1/gazebo/hip_visual.stl"/>
         </geometry>
-      </collision>
-      <visual>
-        <origin xyz="0 0 0" rpy="0 0 0"/>
-        <geometry>
-          <mesh filename="package://legs_description/meshes/iteration_1/gazebo/hip_visual.stl"/>
-        </geometry>
-        <material name="orange"/>
-      </visual>
-      <inertial>
-        <origin xyz="0 0 0" rpy="0 0 0"/>
-        <mass value="0.01"/>
-        <inertia
-          ixx="0.01" ixy="0.0" ixz="0.0"
-          iyy="0.01" iyz="0.0"
-          izz="0.01"/>
+        <material name="orange"/>
+      </visual>
+      <inertial>
+        <origin xyz="0 0 0" rpy="0 0 0"/>
+        <mass value="0.156"/>
+        <inertia
+          ixx="3.03e-004" ixy="0.0" ixz="1.44e-008"
+          iyy="2.78e-005" iyz="0.0"
+          izz="3.14e-004"/>
       </inertial>
     </link>
     <link name="left_upper_limb">
       <collision>
+        <origin xyz="0 0.131 0" rpy="${90*DEG_TO_RAD} 0 0"/>
+        <geometry>
+          <cylinder length="0.262" radius="0.01"/>
+        </geometry>
+      </collision>
+      <visual>
         <origin xyz="0 0 0" rpy="0 0 0"/>
         <geometry>
           <mesh filename="package://legs_description/meshes/iteration_1/gazebo/left_upper_limb_visual.stl"/>
         </geometry>
-      </collision>
-      <visual>
-        <origin xyz="0 0 0" rpy="0 0 0"/>
-        <geometry>
-          <mesh filename="package://legs_description/meshes/iteration_1/gazebo/left_upper_limb_visual.stl"/>
-        </geometry>
-        <material name="orange"/>
-      </visual>
-      <inertial>
-        <origin xyz="0 0 0" rpy="0 0 0"/>
-        <mass value="0.01"/>
-        <inertia
-          ixx="0.01" ixy="0.0" ixz="0.0"
-          iyy="0.01" iyz="0.0"
-          izz="0.01"/>
+        <material name="orange"/>
+      </visual>
+      <inertial>
+        <origin xyz="0 0 0" rpy="90 0 0"/>
+        <mass value="0.123"/>
+        <inertia
+          ixx="1.19e-003" ixy="2.89e-006" ixz="-1.36e-008"
+          iyy="1.69e-005" iyz="-1.78e-005"
+          izz="1.18e-003"/>
       </inertial>
     </link>
     <link name="left_lower_limb">
       <collision>
+        <origin xyz="0 0.131 0" rpy="${90*DEG_TO_RAD} 0 0"/>
+        <geometry>
+          <cylinder length="0.212" radius="0.01"/>
+        </geometry>
+      </collision>
+      <visual>
         <origin xyz="0 0 0" rpy="0 0 0"/>
         <geometry>
           <mesh filename="package://legs_description/meshes/iteration_1/gazebo/left_lower_limb_visual.stl"/>
         </geometry>
-      </collision>
-      <visual>
-        <origin xyz="0 0 0" rpy="0 0 0"/>
-        <geometry>
-          <mesh filename="package://legs_description/meshes/iteration_1/gazebo/left_lower_limb_visual.stl"/>
-        </geometry>
-        <material name="orange"/>
-      </visual>
-      <inertial>
-        <origin xyz="0 0 0" rpy="0 0 0"/>
-        <mass value="0.01"/>
-        <inertia
-          ixx="0.01" ixy="0.0" ixz="0.0"
-          iyy="0.01" iyz="0.0"
-          izz="0.01"/>
+        <material name="orange"/>
+      </visual>
+      <inertial>
+        <origin xyz="0 0 0" rpy="0 0 0"/>
+        <mass value="0.115"/>
+        <inertia
+          ixx="6.99e-004" ixy="2.44e-005" ixz="0.0"
+          iyy="1.85e-005" iyz="-1.82e-005"
+          izz="6.94e-004"/>
       </inertial>
     </link>
@@ -160,55 +120,55 @@
       <inertial>
         <origin xyz="0 0 0" rpy="0 0 0"/>
-        <mass value="0.01"/>
-        <inertia
-          ixx="0.01" ixy="0.0" ixz="0.0"
-          iyy="0.01" iyz="0.0"
-          izz="0.01"/>
+        <mass value="0.021"/>
+        <inertia
+          ixx="2.2e-005" ixy="-9.16e-006" ixz="0.0"
+          iyy="-9.16e-006" iyz="9.05e-006"
+          izz="2.88e-005"/>
       </inertial>
     </link>
     <link name="right_upper_limb">
       <collision>
+        <origin xyz="0 0.131 0" rpy="${90*DEG_TO_RAD} 0 0"/>
+        <geometry>
+          <cylinder length="0.262" radius="0.01"/>
+        </geometry>
+      </collision>
+      <visual>
         <origin xyz="0 0 0" rpy="0 0 0"/>
         <geometry>
           <mesh filename="package://legs_description/meshes/iteration_1/gazebo/right_upper_limb_visual.stl"/>
         </geometry>
-      </collision>
-      <visual>
-        <origin xyz="0 0 0" rpy="0 0 0"/>
-        <geometry>
-          <mesh filename="package://legs_description/meshes/iteration_1/gazebo/right_upper_limb_visual.stl"/>
-        </geometry>
-        <material name="orange"/>
-      </visual>
-      <inertial>
-        <origin xyz="0 0 0" rpy="0 0 0"/>
-        <mass value="0.01"/>
-        <inertia
-          ixx="0.01" ixy="0.0" ixz="0.0"
-          iyy="0.01" iyz="0.0"
-          izz="0.01"/>
+        <material name="orange"/>
+      </visual>
+      <inertial>
+        <origin xyz="0 0 0" rpy="0 0 0"/>
+        <mass value="0.123"/>
+        <inertia
+          ixx="1.19e-003" ixy="2.89e-006" ixz="-1.36e-008"
+          iyy="1.69e-005" iyz="-1.78e-005"
+          izz="1.18e-003"/>
       </inertial>
     </link>
     <link name="right_lower_limb">
       <collision>
+        <origin xyz="0 0.131 0" rpy="${90*DEG_TO_RAD} 0 0"/>
+        <geometry>
+          <cylinder length="0.212" radius="0.01"/>
+        </geometry>
+      </collision>
+      <visual>
         <origin xyz="0 0 0" rpy="0 0 0"/>
         <geometry>
           <mesh filename="package://legs_description/meshes/iteration_1/gazebo/right_lower_limb_visual.stl"/>
         </geometry>
-      </collision>
-      <visual>
-        <origin xyz="0 0 0" rpy="0 0 0"/>
-        <geometry>
-          <mesh filename="package://legs_description/meshes/iteration_1/gazebo/right_lower_limb_visual.stl"/>
-        </geometry>
-        <material name="orange"/>
-      </visual>
-      <inertial>
-        <origin xyz="0 0 0" rpy="0 0 0"/>
-        <mass value="0.01"/>
-        <inertia
-          ixx="0.01" ixy="0.0" ixz="0.0"
-          iyy="0.01" iyz="0.0"
-          izz="0.01"/>
+        <material name="orange"/>
+      </visual>
+      <inertial>
+        <origin xyz="0 0 0" rpy="0 0 0"/>
+        <mass value="0.115"/>
+        <inertia
+          ixx="6.99e-004" ixy="2.44e-005" ixz="0.0"
+          iyy="1.85e-005" iyz="-1.82e-005"
+          izz="6.94e-004"/>
       </inertial>
     </link>
@@ -229,9 +189,9 @@
       <inertial>
         <origin xyz="0 0 0" rpy="0 0 0"/>
-        <mass value="0.01"/>
-        <inertia
-          ixx="0.01" ixy="0.0" ixz="0.0"
-          iyy="0.01" iyz="0.0"
-          izz="0.01"/>
+        <mass value="0.021"/>
+        <inertia
+          ixx="2.2e-005" ixy="-9.16e-006" ixz="0.0"
+          iyy="-9.16e-006" iyz="9.05e-006"
+          izz="2.88e-005"/>
       </inertial>
     </link>
@@ -240,30 +200,32 @@
   -->
   <link name="world"/>
-<!--   <link name="plane_x">
+<!--   <link name="world_pris">
     <inertial>
       <mass value="2e-06"/>
       <inertia ixx="1.1e-09" ixy="0" ixz="0" iyy="1.1e-09" iyz="0" izz="1.1e-09"/>
     </inertial>
-  </link> -->
+  </link>
+  <joint name="world_world_pris" type="prismatic">
+    <origin xyz="0 0 1" rpy="0 0 0"/>
+    <parent link="world"/>
+    <child link="world_pris"/>
+    <axis xyz="0 0 1"/>
+    <limit effort="1000" velocity="1000" lower="0" upper="5" />
+  </joint>
+  <joint name="world_pris_hip" type="continuous">
+    <origin xyz="0 0 0" rpy="0 0 0"/>
+    <parent link="world_pris"/>
+    <child link="hip"/>
+    <axis xyz="0 1 0"/>
+  </joint> -->
+<!--
+  <joint name="world_hip" type="continuous">
+    <origin xyz="0 0 1" rpy="0 0 0"/>
+    <parent link="world"/>
+    <child link="hip"/>
+  </joint>  -->
 	<!--
 		Joints
 	-->
-<!--   <joint name="world_plane_x" type="planar">
-    <parent link="world"/>
-    <child link="plane_x"/>
-    <origin xyz="0 0 1" rpy="0 0 0"/>
-    <axis xyz="1 0 0"/>
-  </joint>
-  <joint name="plane_x_body" type="continuous">
-    <parent link="plane_x"/>
-    <child link="hip"/>
-    <origin xyz="0 0 0" rpy="0 0 0"/>
-    <axis xyz="1 0 0"/>
-  </joint>  -->
-  <joint name="world_hip" type="fixed">
-    <parent link="world"/>
-    <child link="hip"/>
-    <origin xyz="0 0 1" rpy="0 0 0"/>
-  </joint>
   <joint name="left_hip" type="revolute">
     <parent link="hip"/>
@@ -272,5 +234,5 @@
     <axis xyz="0 0 -1"/>
     <limit effort="${upperLegLimitEffort}" velocity="${upperLegLimitVelocity}" lower="${upperLegLimitLowerPosition*DEG_TO_RAD}" upper="${upperLegLimitUpperPosition*DEG_TO_RAD}" />
-    <dynamics damping="${upperLegDamping}"/>
+    <dynamics damping="${damping}"/>
   </joint>
   <joint name="left_knee" type="revolute">
@@ -280,5 +242,5 @@
     <axis xyz="0 0 -1"/>
     <limit effort="${lowerLegLimitEffort}" velocity="${lowerLegLimitVelocity}" lower="${lowerLegLimitLowerPosition*DEG_TO_RAD}" upper="${lowerLegLimitUpperPosition*DEG_TO_RAD}" />
-    <dynamics damping="${lowerLegDamping}"/>
+    <dynamics damping="${damping}"/>
   </joint>
   <joint name="left_ankle" type="revolute">
@@ -288,5 +250,5 @@
     <axis xyz="0 0 -1"/>
     <limit effort="${footLimitEffort}" velocity="${footLimitVelocity}" lower="${footLimitLowerPosition*DEG_TO_RAD}" upper="${footLimitUpperPosition*DEG_TO_RAD}" />
-    <dynamics damping="${footDamping}"/>
+    <dynamics damping="${damping}"/>
   </joint>
   <joint name="right_hip" type="revolute">
@@ -296,5 +258,5 @@
     <axis xyz="0 0 -1"/>
     <limit effort="${upperLegLimitEffort}" velocity="${upperLegLimitVelocity}" lower="${upperLegLimitLowerPosition*DEG_TO_RAD}" upper="${upperLegLimitUpperPosition*DEG_TO_RAD}" />
-    <dynamics damping="${upperLegDamping}"/>
+    <dynamics damping="${damping}"/>
   </joint>
   <joint name="right_knee" type="revolute">
@@ -304,5 +266,5 @@
     <axis xyz="0 0 -1"/>
     <limit effort="${lowerLegLimitEffort}" velocity="${lowerLegLimitVelocity}" lower="${lowerLegLimitLowerPosition*DEG_TO_RAD}" upper="${lowerLegLimitUpperPosition*DEG_TO_RAD}" />
-    <dynamics damping="${lowerLegDamping}"/>
+    <dynamics damping="${damping}"/>
   </joint>
   <joint name="right_ankle" type="revolute">
@@ -312,5 +274,5 @@
     <axis xyz="0 0 -1"/>
     <limit effort="${footLimitEffort}" velocity="${footLimitVelocity}" lower="${footLimitLowerPosition*DEG_TO_RAD}" upper="${footLimitUpperPosition*DEG_TO_RAD}" />
-    <dynamics damping="${footDamping}"/>
+    <dynamics damping="${damping}"/>
   </joint>
   <transmission name="left_hip_trans">
@@ -374,3 +336,110 @@
     </actuator>
   </transmission>
+  <!-- Rotational robot holder -->
+  <xacro:property name="rotational_robot_holder_base_length_extra" value="0" />
+  <xacro:if value="${robot_floating is 1}">
+    <xacro:property name="rotational_robot_holder_base_length_extra" value="0.1" />
+  </xacro:if>
+  <xacro:property name="rotational_robot_holder_base_length" value="1" />
+  <xacro:property name="rotational_robot_holder_base_radius" value="0.2" />
+  <xacro:property name="rotational_robot_holder_holder_radius" value="0.01" />
+  <xacro:property name="rotational_robot_holder_holder_length" value="2" />
+  <!-- <xacro:include filename="$(find gazebo_resources)/models/rotational_robot_holder/urdf/rotational_robot_holder.xacro" /> -->
+  <link name="rotational_robot_holder_base">
+    <collision>
+      <origin xyz="0 0 0" rpy="0 0 0"/>
+      <geometry>
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
Commit message: updated

File: src/legs_description/urdf/legs.urdf (robot description, URDF)
Before this commit: robot legs, 11 links, 10 joints
Links:
- link hip: mass 0.156 -> 9.984; geometry collision cylinder length=0.72 radius=0.1; visual mesh filename=package://legs_description/meshes/iteration_1/gazebo/hip_vi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 scale=4 4 4
- link left_foot: mass 0.021 -> 1.344; geometry collision mesh filename=package://legs_description/meshes/iteration_1/gazebo/left_f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 scale=4 4 4; visual mesh filename=package://legs_description/meshes/iteration_1/gazebo/left_f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 scale=4 4 4
- link left_lower_limb: mass 0.115 -> 7.36; geometry collision cylinder length=0.848 radius=0.04; visual mesh filename=package://legs_description/meshes/iteration_1/gazebo/left_l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 scale=4 4 4
- link left_upper_limb: mass 0.123 -> 7.872; geometry collision cylinder length=1.048 radius=0.04; visual mesh filename=package://legs_description/meshes/iteration_1/gazebo/left_u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 scale=4 4 4
- link right_foot: mass 0.021 -> 1.344; geometry collision mesh filename=package://legs_description/meshes/iteration_1/gazebo/right_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 scale=4 4 4; visual mesh filename=package://legs_description/meshes/iteration_1/gazebo/right_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 scale=4 4 4
- link right_lower_limb: mass 0.115 -> 7.36; geometry collision cylinder length=0.848 radius=0.04; visual mesh filename=package://legs_description/meshes/iteration_1/gazebo/right_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 scale=4 4 4
- link right_upper_limb: mass 0.123 -> 7.872; geometry collision cylinder length=1.048 radius=0.04; visual mesh filename=package://legs_description/meshes/iteration_1/gazebo/right_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 scale=4 4 4
- link rotational_robot_holder_base: geometry collision cylinder length=2.68 radius=0.8; visual cylinder length=2.68 radius=0.8
- link rotational_robot_holder_holder: geometry collision cylinder length=8 radius=0.04; visual cylinder length=8 radius=0.04
- link rotational_robot_holder_virtual: mass 0.01 -> $0.01
Joints:
- joint left_ankle: origin xyz=0 0.212 0 rpy=0 0 0 -> xyz=0 0.848 0 rpy=0 0 0
- joint left_hip: origin xyz=0 0.0635 -0.028867 rpy=-1.57079632679 0 0 -> xyz=0 0.254 -0.115468 rpy=-1.57079632679 0 0
- joint left_knee: origin xyz=0 0.262 0 rpy=0 0 0 -> xyz=0 1.048 0 rpy=0 0 0
- joint right_ankle: origin xyz=0 0.212 0 rpy=0 0 0 -> xyz=0 0.848 0 rpy=0 0 0
- joint right_hip: origin xyz=0 -0.0635 -0.028867 rpy=-1.57079632679 0 0 -> xyz=0 -0.254 -0.115468 rpy=-1.57079632679 0 0
- joint right_knee: origin xyz=0 0.262 0 rpy=0 0 0 -> xyz=0 1.048 0 rpy=0 0 0
- joint rotational_robot_holder_base_to_world: origin xyz=0 0 0.5 rpy=0 0 0 -> xyz=0 0 1.34 rpy=0 0 0
- joint rotational_robot_holder_joint: origin xyz=0 0 0.5 rpy=0 0 0 -> xyz=0 0 1.34 rpy=0 0 0
- joint rotational_robot_holder_to_rotot: origin xyz=2.2 0 0 rpy=0 0 0 -> xyz=8.2 0 0 rpy=0 0 0
