Commit message: removed inertias under 1e-005

File: src/legs_description/urdf/legs.urdf (robot description, URDF)
Before this commit: robot legs, 11 links, 10 joints
Links:
- link hip: mass 9.984 -> 0.156; geometry collision cylinder length=0.18 radius=0.025; visual mesh filename=package://legs_description/meshes/iteration_1/gazebo/hip_vi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 scale=1 1 1
- link left_foot: mass 1.344 -> 0.021; geometry collision mesh filename=package://legs_description/meshes/iteration_1/gazebo/left_f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 scale=1 1 1; visual mesh filename=package://legs_description/meshes/iteration_1/gazebo/left_f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 scale=1 1 1
- link left_lower_limb: mass 7.36 -> 0.115; geometry collision cylinder length=0.212 radius=0.01; visual mesh filename=package://legs_description/meshes/iteration_1/gazebo/left_l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 scale=1 1 1
- link left_upper_limb: mass 7.872 -> 0.123; geometry collision cylinder length=0.262 radius=0.01; visual mesh filename=package://legs_description/meshes/iteration_1/gazebo/left_u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 scale=1 1 1
- link right_foot: mass 1.344 -> 0.021; geometry collision mesh filename=package://legs_description/meshes/iteration_1/gazebo/right_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 scale=1 1 1; visual mesh filename=package://legs_description/meshes/iteration_1/gazebo/right_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 scale=1 1 1
- link right_lower_limb: mass 7.36 -> 0.115; geometry collision cylinder length=0.212 radius=0.01; visual mesh filename=package://legs_description/meshes/iteration_1/gazebo/right_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 scale=1 1 1
- link right_upper_limb: mass 7.872 -> 0.123; geometry collision cylinder length=0.262 radius=0.01; visual mesh filename=package://legs_description/meshes/iteration_1/gazebo/right_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 scale=1 1 1
- link rotational_robot_holder_base: geometry collision cylinder length=0.67 radius=0.2; visual cylinder length=0.67 radius=0.2
- link rotational_robot_holder_holder: mass 0.01 -> 0.001; geometry collision cylinder length=2 radius=0.01; visual cylinder length=2 radius=0.01
- link rotational_robot_holder_virtual: mass $0.01 -> 0.001
Joints:
- joint left_ankle: origin xyz=0 0.848 0 rpy=0 0 0 -> xyz=0 0.212 0 rpy=0 0 0
- joint left_hip: origin xyz=0 0.254 -0.115468 rpy=-1.57079632679 0 0 -> xyz=0 0.0635 -0.028867 rpy=-1.57079632679 0 0
- joint left_knee: origin xyz=0 1.048 0 rpy=0 0 0 -> xyz=0 0.262 0 rpy=0 0 0
- joint right_ankle: origin xyz=0 0.848 0 rpy=0 0 0 -> xyz=0 0.212 0 rpy=0 0 0
- joint right_hip: origin xyz=0 -0.254 -0.115468 rpy=-1.57079632679 0 0 -> xyz=0 -0.0635 -0.028867 rpy=-1.57079632679 0 0
- joint right_knee: origin xyz=0 1.048 0 rpy=0 0 0 -> xyz=0 0.262 0 rpy=0 0 0
- joint rotational_robot_holder_base_to_world: origin xyz=0 0 1.34 rpy=0 0 0 -> xyz=0 0 0.335 rpy=0 0 0
- joint rotational_robot_holder_joint: origin xyz=0 0 1.34 rpy=0 0 0 -> xyz=0 0 0.335 rpy=0 0 0
- joint rotational_robot_holder_to_rotot: limit lower=0 upper=1 effort=30 velocity=1.0 -> lower=0 upper=1 effort=30 velocity=2.0; origin xyz=8.2 0 0 rpy=0 0 0 -> xyz=2.02 0 0 rpy=0 0 1.57079632679

File: src/legs_description/urdf/legs.xacro (robot description, xacro)
@@ -5,9 +5,9 @@
 	<xacro:property name="DEG_TO_RAD" value="${PI/180}"/>
 	<!-- ROS -->
-	<xacro:property name="update_rate" value="10"/>
+	<xacro:property name="update_rate" value="1"/>
 	<xacro:property name="robot_name" value="legs"/>
   <!-- Robot configuration: Miscellaneous -->
   <xacro:property name="robot_floating" value="0"/>
-  <xacro:property name="scale" value="10"/>
+  <xacro:property name="scale" value="1"/>
   <xacro:property name="mass_scale" value="${pow(scale,3)}"/>
   <xacro:property name="intertia_scale" value="${pow(scale,1.667)}"/>
@@ -15,5 +15,5 @@
 	<xacro:property name="max_real_motor_torque" value="1.0787315"/> <!-- In N*m -->
   <!-- Robot configuration: Geometry -->
-  <xacro:property name="damping" value="0.7" />
+  <xacro:property name="damping" value="0.1" />
   <xacro:property name="upperLegHeight" value="0.262" />
   <xacro:property name="upperLegDiameter" value="0.02" />
@@ -56,6 +56,6 @@
         <mass value="${mass_scale*0.156}"/>
         <inertia
-          ixx="${intertia_scale*3.03e-004}" ixy="${intertia_scale*0.0}" ixz="${intertia_scale*1.44e-008}"
-          iyy="${intertia_scale*2.78e-005}" iyz="${intertia_scale*0.0}"
+          ixx="${intertia_scale*3.03e-004}" ixy="0.0" ixz="0.0"
+          iyy="0.0" iyz="0.0"
           izz="${intertia_scale*3.14e-004}"/>
       </inertial>
@@ -79,6 +79,6 @@
         <mass value="${mass_scale*0.123}"/>
         <inertia
-          ixx="${intertia_scale*1.19e-003}" ixy="${intertia_scale*2.89e-006}" ixz="${intertia_scale*-1.36e-008}"
-          iyy="${intertia_scale*1.69e-005}" iyz="${intertia_scale*-1.78e-005}"
+          ixx="${intertia_scale*1.19e-003}" ixy="0.0" ixz="0.0"
+          iyy="0.0" iyz="0.0"
           izz="${intertia_scale*1.18e-003}"/>
       </inertial>
@@ -102,6 +102,6 @@
         <mass value="${mass_scale*0.115}"/>
         <inertia
-          ixx="${intertia_scale*6.99e-004}" ixy="${intertia_scale*2.44e-005}" ixz="${intertia_scale*0.0}"
-          iyy="${intertia_scale*1.85e-005}" iyz="${intertia_scale*-1.82e-005}"
+          ixx="${intertia_scale*6.99e-004}" ixy="0.0" ixz="0.0"
+          iyy="0.0" iyz="0.0"
           izz="${intertia_scale*6.94e-004}"/>
       </inertial>
@@ -125,7 +125,7 @@
         <mass value="${mass_scale*0.021}"/>
         <inertia
-          ixx="${intertia_scale*2.2e-005}" ixy="${intertia_scale*-9.16e-006}" ixz="${intertia_scale*0.0}"
-          iyy="${intertia_scale*-9.16e-006}" iyz="${intertia_scale*9.05e-006}"
-          izz="${intertia_scale*2.88e-005}"/>
+          ixx="0.0" ixy="0.0" ixz="0.0"
+          iyy="0.0" iyz="0.0"
+          izz="0.0"/>
       </inertial>
     </link>
@@ -148,6 +148,6 @@
         <mass value="${mass_scale*0.123}"/>
         <inertia
-          ixx="${intertia_scale*1.19e-003}" ixy="${intertia_scale*2.89e-006}" ixz="${intertia_scale*-1.36e-008}"
-          iyy="${intertia_scale*1.69e-005}" iyz="${intertia_scale*-1.78e-005}"
+          ixx="${intertia_scale*1.19e-003}" ixy="0.0" ixz="0.0"
+          iyy="0.0" iyz="0.0"
           izz="${intertia_scale*1.18e-003}"/>
       </inertial>
@@ -171,6 +171,6 @@
         <mass value="${mass_scale*0.115}"/>
         <inertia
-          ixx="${intertia_scale*6.99e-004}" ixy="${intertia_scale*2.44e-005}" ixz="${intertia_scale*0.0}"
-          iyy="${intertia_scale*1.85e-005}" iyz="${intertia_scale*-1.82e-005}"
+          ixx="${intertia_scale*6.99e-004}" ixy="0.0" ixz="0.0"
+          iyy="0.0" iyz="0.0"
           izz="${intertia_scale*6.94e-004}"/>
       </inertial>
@@ -194,6 +194,6 @@
         <mass value="${mass_scale*0.021}"/>
         <inertia
-          ixx="${intertia_scale*2.2e-005}" ixy="${intertia_scale*-9.16e-006}" ixz="${intertia_scale*0.0}"
-          iyy="${intertia_scale*-9.16e-006}" iyz="${intertia_scale*9.05e-006}"
+          ixx="${intertia_scale*2.2e-005}" ixy="0.0" ixz="0.0"
+          iyy="0.0" iyz="0.0"
           izz="${intertia_scale*2.88e-005}"/>
       </inertial>
@@ -382,5 +382,5 @@
     </visual>
     <inertial>
-      <mass value="0.01"/>
+      <mass value="0.001"/>
       <inertia ixx="0.002" ixy="0.0" ixz="0.0" iyy="0.002" iyz="0.0" izz="0.002"/>
     </inertial>
@@ -401,5 +401,5 @@
     </visual>
     <inertial>
-      <mass value="0.01"/>
+      <mass value="0.001"/>
       <inertia ixx="0.002" ixy="0.0" ixz="0.0" iyy="0.002" iyz="0.0" izz="0.002"/>
     </inertial>
@@ -427,5 +427,4 @@
       <origin xyz="0 0 0" rpy="0 0 0"/>
       <axis xyz="0 1 0"/>
-      <dynamics damping="0.7"/>
     </joint>
     <joint name="rotational_robot_holder_joint" type="continuous">
@@ -434,5 +433,4 @@
       <origin xyz="0 0 ${rotational_robot_holder_base_length/2}" rpy="0 0 0"/>
       <axis xyz="0 0 1"/>
-      <dynamics damping="0.7"/>
     </joint>
   </xacro:if>
@@ -440,7 +438,7 @@
     <parent link="rotational_robot_holder_holder"/>
     <child link="hip"/>
-    <origin xyz="${rotational_robot_holder_holder_length+0.2} 0 0" rpy="0 0 0"/>
+    <origin xyz="${rotational_robot_holder_holder_length+0.2} 0 0" rpy="0 0 ${90*DEG_TO_RAD}"/>
     <axis xyz="0 0 1"/>
-    <limit effort="30" velocity="1.0" lower="0" upper="1" />
+    <limit effort="30" velocity="2.0" lower="0" upper="1" />
   </joint>
 </robot>
