Commit message: updated values to iteration 1

File: src/legs_description/urdf/legs.xacro (robot description, xacro)
@@ -18,15 +18,7 @@
   <xacro:property name="scale" value="1" />
   <xacro:property name="minimum_intertia" value="0.002" /> <!-- <0.001 doesn't work -->
-	<xacro:property name="bodyWidth" value="${0.085*scale}" />
-	<xacro:property name="bodyLength" value="${0.08*scale}" />
-	<xacro:property name="bodyHeight" value="${0.065*scale}" />
-	<xacro:property name="bodyMass" value="${0.45*scale}" />
-	<xacro:property name="weightWidth" value="${0.05*scale}" />
-	<xacro:property name="weightLength" value="${0.07*scale}" />
-	<xacro:property name="weightHeight" value="${0.025*scale}" />
-	<xacro:property name="weightMass" value="${0.50*scale}" />
 	<xacro:property name="upperLegWidth" value="${0.015*scale}" />
 	<xacro:property name="upperLegLength" value="${0.015*scale}" />
-	<xacro:property name="upperLegHeight" value="${0.142*scale}" />
+	<xacro:property name="upperLegHeight" value="${0.262*scale}" />
 	<xacro:property name="upperLegMass" value="${0.163*scale}" />
   <xacro:property name="upperLegLimitUpperPosition" value="30" />
@@ -37,5 +29,5 @@
 	<xacro:property name="lowerLegWidth" value="${0.015*scale}" />
 	<xacro:property name="lowerLegLength" value="${0.015*scale}" />
-	<xacro:property name="lowerLegHeight" value="${0.125*scale}" />
+	<xacro:property name="lowerLegHeight" value="${0.212*scale}" />
 	<xacro:property name="lowerLegMass" value="${0.17*scale}" />
   <xacro:property name="lowerLegLimitUpperPosition" value="0" />
@@ -45,5 +37,5 @@
   <xacro:property name="lowerLegDamping" value="0.7" />
 	<xacro:property name="footWidth" value="${0.015*scale}" />
-	<xacro:property name="footLength" value="${0.050*scale}" />
+	<xacro:property name="footLength" value="${0.095*scale}" />
 	<xacro:property name="footHeight" value="${0.008*scale}" />
 	<xacro:property name="footMass" value="${0.0296*scale}" />
@@ -53,5 +45,13 @@
   <xacro:property name="footLimitEffort" value="10" />
   <xacro:property name="footDamping" value="0.7" />
-	<xacro:property name="legDistFromCenter" value="${0.015*scale}" />
+	<xacro:property name="legDistFromCenter" value="${0.075*scale}" />
+  <xacro:property name="bodyWidth" value="${legDistFromCenter*2+0.02*scale}" />
+  <xacro:property name="bodyLength" value="${0.08*scale}" />
+  <xacro:property name="bodyHeight" value="${0.065*scale}" />
+  <xacro:property name="bodyMass" value="${0.45*scale}" />
+  <xacro:property name="weightWidth" value="${0.05*scale}" />
+  <xacro:property name="weightLength" value="${0.07*scale}" />
+  <xacro:property name="weightHeight" value="${0.025*scale}" />
+  <xacro:property name="weightMass" value="${0.50*scale}" />
 	<xacro:property name="footAnklePos" value="${0.015*scale}" />
 	<xacro:property name="legAnklePos" value="${0*scale}" />

Commit message: added node and service to restart simulation and start with the init positions

File: src/legs_description/urdf/legs.xacro (robot description, xacro)
@@ -40,6 +40,6 @@
 	<xacro:property name="footHeight" value="${0.008*scale}" />
 	<xacro:property name="footMass" value="${0.0296*scale}" />
-  <xacro:property name="footLimitUpperPosition" value="0" />
-  <xacro:property name="footLimitLowerPosition" value="0" />
+  <xacro:property name="footLimitUpperPosition" value="40" />
+  <xacro:property name="footLimitLowerPosition" value="-50" />
   <xacro:property name="footLimitVelocity" value="10" />
   <xacro:property name="footLimitEffort" value="10" />

Commit message: adjusted link limits

File: src/legs_description/urdf/legs.xacro (robot description, xacro)
@@ -22,6 +22,6 @@
 	<xacro:property name="upperLegHeight" value="${0.262*scale}" />
 	<xacro:property name="upperLegMass" value="${0.163*scale}" />
-  <xacro:property name="upperLegLimitUpperPosition" value="30" />
-  <xacro:property name="upperLegLimitLowerPosition" value="-30" />
+  <xacro:property name="upperLegLimitUpperPosition" value="80" />
+  <xacro:property name="upperLegLimitLowerPosition" value="-80" />
   <xacro:property name="upperLegLimitVelocity" value="10" />
   <xacro:property name="upperLegLimitEffort" value="10" />
@@ -40,6 +40,6 @@
 	<xacro:property name="footHeight" value="${0.008*scale}" />
 	<xacro:property name="footMass" value="${0.0296*scale}" />
-  <xacro:property name="footLimitUpperPosition" value="40" />
-  <xacro:property name="footLimitLowerPosition" value="-50" />
+  <xacro:property name="footLimitUpperPosition" value="38" />
+  <xacro:property name="footLimitLowerPosition" value="-52" />
   <xacro:property name="footLimitVelocity" value="10" />
   <xacro:property name="footLimitEffort" value="10" />

Commit message: fixed bugs when creating the limits of the feeet

File: src/legs_description/urdf/legs.xacro (robot description, xacro)
@@ -171,5 +171,5 @@
 		<origin xyz="${lowerLegHeight} 0 0" rpy="0 0 0"/>
 		<axis xyz="0 0 1"/>
-		<limit effort="${footLimitEffort}" velocity="${footLimitVelocity}" lower="${footLimitLowerPosition}" upper="${footLimitUpperPosition}" />
+		<limit effort="${footLimitEffort}" velocity="${footLimitVelocity}" lower="${footLimitLowerPosition*DEG_TO_RAD}" upper="${footLimitUpperPosition*DEG_TO_RAD}" />
 		<dynamics damping="${footDamping}"/>
 	</joint>
@@ -195,5 +195,5 @@
 		<origin xyz="${lowerLegHeight} 0 0" rpy="0 0 0"/>
 		<axis xyz="0 0 1"/>
-		<limit effort="${footLimitEffort}" velocity="${footLimitVelocity}" lower="${footLimitLowerPosition}" upper="${footLimitUpperPosition}" />
+		<limit effort="${footLimitEffort}" velocity="${footLimitVelocity}" lower="${footLimitLowerPosition*DEG_TO_RAD}" upper="${footLimitUpperPosition*DEG_TO_RAD}" />
     <dynamics damping="${footDamping}"/>
 	</joint>

Commit message: switched from rotational holder to virtual joints

File: src/legs_description/urdf/legs.xacro (robot description, xacro)
@@ -141,13 +141,29 @@
 	-->
 	<xacro:create_box name="body" origin_x="0" origin_y="0" origin_z="${bodyHeight/2}" r="0" p="0" y="0" width="${bodyWidth}" length="${bodyLength}" height="${bodyHeight}" mass="${bodyMass}"  />
+  <!--
+    Virtual links
+  -->
+  <link name="world"/>
+  <link name="plane_x">
+    <inertial>
+      <mass value="2e-06"/>
+      <inertia ixx="1.1e-09" ixy="0" ixz="0" iyy="1.1e-09" iyz="0" izz="1.1e-09"/>
+    </inertial>
+  </link>
 	<!--
 		Joints
 	-->
-  <link name="world"/>
-<!--   <joint name="fixed" type="fixed">
+  <joint name="world_plane_x" type="planar">
     <parent link="world"/>
+    <child link="plane_x"/>
+    <origin xyz="0 0 ${footHeight + lowerLegHeight + upperLegHeight}" rpy="0 0 0"/>
+    <axis xyz="1 0 0"/>
+  </joint>
+  <joint name="plane_x_body" type="continuous">
+    <parent link="plane_x"/>
     <child link="body"/>
-    <origin xyz="0 0 ${(footHeight + lowerLegHeight + upperLegHeight)*1.1}" rpy="0 0 0"/>
-  </joint>  -->
+    <origin xyz="0 0 0" rpy="0 0 0"/>
+    <axis xyz="1 0 0"/>
+  </joint>
 	<joint name="left_hip" type="revolute">
 		<parent link="body"/>
@@ -259,4 +275,5 @@
 	</transmission>
 	<!-- Rotational robot holder -->
+<!--
   <xacro:property name="rotational_robot_holder_base_length_extra" value="0" />
   <xacro:if value="${robot_floating is 1}">
@@ -267,5 +284,4 @@
   <xacro:property name="rotational_robot_holder_holder_radius" value="${0.01*scale}" />
   <xacro:property name="rotational_robot_holder_holder_length" value="${2*scale}" />
-	<!-- <xacro:include filename="$(find gazebo_resources)/models/rotational_robot_holder/urdf/rotational_robot_holder.xacro" /> -->
   <link name="rotational_robot_holder_base">
     <collision>
@@ -325,5 +341,4 @@
     </inertial>
   </link>
-  <!-- Robot to rotational_robot_holder -->
   <joint name="rotational_robot_holder_base_to_world" type="fixed">
     <parent link="world"/>
@@ -365,3 +380,4 @@
     <limit effort="30" velocity="1.0" lower="0" upper="1" />
   </joint>
+ -->
 </robot>
