Commit message: added links from solidoworks. The model loads in gazebo and rviz

File: src/legs_description/urdf/legs.xacro (robot description, xacro)
@@ -18,53 +18,35 @@
   <xacro:property name="scale" value="1" />
   <xacro:property name="minimum_intertia" value="0.002" /> <!-- <0.001 doesn't work -->
-	<xacro:property name="upperLegWidth" value="${0.015*scale}" />
-	<xacro:property name="upperLegLength" value="${0.015*scale}" />
-	<xacro:property name="upperLegHeight" value="${0.262*scale}" />
-	<xacro:property name="upperLegMass" value="${0.163*scale}" />
-  <xacro:property name="upperLegLimitUpperPosition" value="80" />
-  <xacro:property name="upperLegLimitLowerPosition" value="-80" />
+  <xacro:property name="upperLegHeight" value="0.262" />
+  <xacro:property name="upperLegDiameter" value="0.02" />
+	<xacro:property name="upperLegMass" value="0.163" />
+  <xacro:property name="upperLegLimitUpperPosition" value="90" />
+  <xacro:property name="upperLegLimitLowerPosition" value="-60" />
   <xacro:property name="upperLegLimitVelocity" value="10" />
   <xacro:property name="upperLegLimitEffort" value="10" />
   <xacro:property name="upperLegDamping" value="0.7" />
-	<xacro:property name="lowerLegWidth" value="${0.015*scale}" />
-	<xacro:property name="lowerLegLength" value="${0.015*scale}" />
-	<xacro:property name="lowerLegHeight" value="${0.212*scale}" />
-	<xacro:property name="lowerLegMass" value="${0.17*scale}" />
+  <xacro:property name="lowerLegHeight" value="0.212" />
+  <xacro:property name="lowerLegDiameter" value="0.02" />
+	<xacro:property name="lowerLegMass" value="0.17" />
   <xacro:property name="lowerLegLimitUpperPosition" value="0" />
-  <xacro:property name="lowerLegLimitLowerPosition" value="-150" />
+  <xacro:property name="lowerLegLimitLowerPosition" value="-120" />
   <xacro:property name="lowerLegLimitVelocity" value="10" />
   <xacro:property name="lowerLegLimitEffort" value="10" />
   <xacro:property name="lowerLegDamping" value="0.7" />
-	<xacro:property name="footWidth" value="${0.015*scale}" />
-	<xacro:property name="footLength" value="${0.095*scale}" />
-	<xacro:property name="footHeight" value="${0.008*scale}" />
-	<xacro:property name="footMass" value="${0.0296*scale}" />
-  <xacro:property name="footLimitUpperPosition" value="38" />
-  <xacro:property name="footLimitLowerPosition" value="-52" />
+	<xacro:property name="footMass" value="0.0296" />
+  <xacro:property name="footLimitUpperPosition" value="120" />
+  <xacro:property name="footLimitLowerPosition" value="-50" />
   <xacro:property name="footLimitVelocity" value="10" />
   <xacro:property name="footLimitEffort" value="10" />
   <xacro:property name="footDamping" value="0.7" />
-	<xacro:property name="legDistFromCenter" value="${0.075*scale}" />
-  <xacro:property name="bodyWidth" value="${legDistFromCenter*2+0.02*scale}" />
-  <xacro:property name="bodyLength" value="${0.08*scale}" />
-  <xacro:property name="bodyHeight" value="${0.065*scale}" />
-  <xacro:property name="bodyMass" value="${0.45*scale}" />
-  <xacro:property name="weightWidth" value="${0.05*scale}" />
-  <xacro:property name="weightLength" value="${0.07*scale}" />
-  <xacro:property name="weightHeight" value="${0.025*scale}" />
-  <xacro:property name="weightMass" value="${0.50*scale}" />
-	<xacro:property name="footAnklePos" value="${0.015*scale}" />
-	<xacro:property name="legAnklePos" value="${0*scale}" />
-	<xacro:property name="lowerKneePos" value="${0.12*scale}" />
-	<xacro:property name="upperKneePos" value="${0.02*scale}" />
-	<xacro:property name="legHipPos" value="${0.132*scale}" />
-	<xacro:property name="bodyHipHeight" value="${0.01*scale}" />
-	<xacro:property name="bodyHipWidth" value="${0.025*scale}" />
-	<xacro:property name="massJointBodyDepth" value="${0.07*scale}" />
-	<xacro:property name="massJointBodyHeight" value="${0.055*scale}" />
-	<xacro:property name="massJointMassDepth" value="${0.065*scale}" />
-	<xacro:property name="massJointMassHeigth" value="${0.007*scale}" />
-	<xacro:property name="armLength" value="${0.6*scale}" />
-	<xacro:property name="armOffset" value="${0.025*scale}" />
+	<xacro:property name="legDistFromCenter" value="0.0635" />
+  <xacro:property name="hipMass" value="${0.45}" />
+	<xacro:property name="footAnklePos" value="${0.015}" />
+	<xacro:property name="legAnklePos" value="${0}" />
+	<xacro:property name="lowerKneePos" value="${0.12}" />
+	<xacro:property name="upperKneePos" value="${0.02}" />
+	<xacro:property name="legHipPos" value="${0.132}" />
+	<xacro:property name="bodyHipHeight" value="${0.01}" />
+	<xacro:property name="bodyHipWidth" value="${0.025}" />
 	<!-- Import Gazebo customizations and colors-->
 	<xacro:include filename="$(find legs_description)/urdf/legs.gazebo" />
@@ -73,46 +55,17 @@
 		Macros
 	 -->
-	 <!-- Box Macro!
-	<xacro:create_box name="" origin_x="" origin_y="" origin_z="" r="" p="" y="" width="" length="" height="" mass=""/>
-	 -->
-	<xacro:macro name="create_box" params="name origin_x origin_y origin_z r p y width length height mass">
-		<!-- Set the minimum intertia -->
-		<xacro:property name="ixx" value="${minimum_intertia}" />
-		<xacro:if value="${mass / 12.0 * (length*length + height*height) > 0.01}">
-			<xacro:property name="ixx" value="${mass / 12.0 * (length*length + height*height)}" />
+		<!-- Intertia Macro: Set the minimum intertia -->
+<!--   <xacro:macro name="check_minimum_intertia" params="inertia">
+		<xacro:if value="${inertia < 0.01}">
+			<xacro:property name="inertia" value="${mass / 12.0 * (3*(diameter/2)^2 + height^2)}" />
 		</xacro:if>
-		<xacro:property name="iyy" value="${minimum_intertia}" />
-		<xacro:if value="${mass / 12.0 * (length*length + height*height) > 0.01}">
-			<xacro:property name="iyy" value="${mass / 12.0 * (length*length + height*height)}" />
-		</xacro:if>
-		<xacro:property name="izz" value="${minimum_intertia}" />
-		<xacro:if value="${mass / 12.0 * (length*length + height*height) > 0.01}">
-			<xacro:property name="izz" value="${mass / 12.0 * (length*length + height*height)}" />
-		</xacro:if>
-		<!-- Creates the link -->
-		<link name="${name}">
-			<collision>
-				<origin xyz="${origin_x} ${origin_y} ${origin_z}" rpy="${r} ${p} ${y}"/>
-				<geometry>
-					<box size="${width} ${length} ${height}" />
-				</geometry>
-			</collision>
-			<visual>
-				<origin xyz="${origin_x} ${origin_y} ${origin_z}" rpy="${r} ${p} ${y}"/>
-				<geometry>
-					<box size="${width} ${length} ${height}" />
-				</geometry>
-				<material name="orange"/>
-			</visual>
-			<inertial>
-				<origin xyz="${origin_x} ${origin_y} ${origin_z}" rpy="${r} ${p} ${y}"/>
-				<mass value="${mass}"/>
-				<inertia
-					ixx="${ixx}" ixy="0.0" ixz="0.0"
-					iyy="${iyy}" iyz="0.0"
-					izz="${izz}"/>
-			</inertial>
-		</link>
+    <xacro:if value="${inertia < 0.01}">
+      <xacro:property name="inertia" value="${mass / 12.0 * (3*(diameter/2)^2 + height^2)}" />
+    </xacro:if>
+    <xacro:if value="${inertia < 0.01}">
+      <xacro:property name="inertia" value="${mass / 12.0 * (3*(diameter/2)^2 + height^2)}" />
+    </xacro:if>
 	</xacro:macro>
+ -->
 	<!--
 		World
@@ -122,262 +75,302 @@
 		Left Leg
 	-->
-	<!-- Left Foot -->
-	<xacro:create_box name="left_foot" origin_x="${footHeight/2}" origin_y="${footLength/2 - footAnklePos}" origin_z="0" r="0" p="${-PI/2}" y="0" width="${footWidth}" length="${footLength}" height="${footHeight}" mass="${footMass}"  />
-	<!-- Left Lower Leg -->
-	<xacro:create_box name="left_lower_leg" origin_x="${lowerLegHeight/2}" origin_y="0" origin_z="0" r="0" p="${-PI/2}" y="0" width="${lowerLegWidth}" length="${lowerLegLength}" height="${lowerLegHeight}" mass="${lowerLegMass}"  />
-	<!-- Left Upper Leg -->
-	<xacro:create_box name="left_upper_leg" origin_x="${upperLegHeight/2}" origin_y="0" origin_z="0" r="0" p="${-PI/2}" y="0" width="${upperLegWidth}" length="${upperLegLength}" height="${upperLegHeight}" mass="${upperLegMass}"   />
-	<!--
-		Right Leg
-	-->
-	<!-- Right Foot -->
-	<xacro:create_box name="right_foot" origin_x="${footHeight/2}" origin_y="${footLength/2 - footAnklePos}" origin_z="0" r="0" p="${-PI/2}" y="0" width="${footWidth}" length="${footLength}" height="${footHeight}" mass="${footMass}"   />
-	<!-- Right Lower Leg -->
-	<xacro:create_box name="right_lower_leg" origin_x="${lowerLegHeight/2}" origin_y="0" origin_z="0" r="0" p="${-PI/2}" y="0" width="${lowerLegWidth}" length="${lowerLegLength}" height="${lowerLegHeight}" mass="${lowerLegMass}"   />
-	<!-- Right Upper Leg -->
-	<xacro:create_box name="right_upper_leg" origin_x="${upperLegHeight/2}" origin_y="0" origin_z="0" r="0" p="${-PI/2}" y="0" width="${upperLegWidth}" length="${upperLegLength}" height="${upperLegHeight}" mass="${upperLegMass}"   />
-	<!--
-		Body
-	-->
-	<xacro:create_box name="body" origin_x="0" origin_y="0" origin_z="${bodyHeight/2}" r="0" p="0" y="0" width="${bodyWidth}" length="${bodyLength}" height="${bodyHeight}" mass="${bodyMass}"  />
+    <link name="hip">
+      <collision>
+        <origin xyz="0 0 0" rpy="0 0 0"/>
+        <geometry>
+          <mesh filename="package://legs_description/meshes/iteration_1/gazebo/hip_visual.stl"/>
+        </geometry>
+      </collision>
+      <visual>
+        <origin xyz="0 0 0" rpy="0 0 0"/>
+        <geometry>
+          <mesh filename="package://legs_description/meshes/iteration_1/gazebo/hip_visual.stl"/>
+        </geometry>
+        <material name="orange"/>
+      </visual>
+      <inertial>
+        <origin xyz="0 0 0" rpy="0 0 0"/>
+        <mass value="0.01"/>
+        <inertia
+          ixx="0.01" ixy="0.0" ixz="0.0"
+          iyy="0.01" iyz="0.0"
+          izz="0.01"/>
+      </inertial>
+    </link>
+    <link name="left_upper_limb">
+      <collision>
+        <origin xyz="0 0 0" rpy="0 0 0"/>
+        <geometry>
+          <mesh filename="package://legs_description/meshes/iteration_1/gazebo/left_upper_limb_visual.stl"/>
+        </geometry>
+      </collision>
+      <visual>
+        <origin xyz="0 0 0" rpy="0 0 0"/>
+        <geometry>
+          <mesh filename="package://legs_description/meshes/iteration_1/gazebo/left_upper_limb_visual.stl"/>
+        </geometry>
+        <material name="orange"/>
+      </visual>
+      <inertial>
+        <origin xyz="0 0 0" rpy="0 0 0"/>
+        <mass value="0.01"/>
+        <inertia
+          ixx="0.01" ixy="0.0" ixz="0.0"
+          iyy="0.01" iyz="0.0"
+          izz="0.01"/>
+      </inertial>
+    </link>
+    <link name="left_lower_limb">
+      <collision>
+        <origin xyz="0 0 0" rpy="0 0 0"/>
+        <geometry>
+          <mesh filename="package://legs_description/meshes/iteration_1/gazebo/left_lower_limb_visual.stl"/>
+        </geometry>
+      </collision>
+      <visual>
+        <origin xyz="0 0 0" rpy="0 0 0"/>
+        <geometry>
+          <mesh filename="package://legs_description/meshes/iteration_1/gazebo/left_lower_limb_visual.stl"/>
+        </geometry>
+        <material name="orange"/>
+      </visual>
+      <inertial>
+        <origin xyz="0 0 0" rpy="0 0 0"/>
+        <mass value="0.01"/>
+        <inertia
+          ixx="0.01" ixy="0.0" ixz="0.0"
+          iyy="0.01" iyz="0.0"
+          izz="0.01"/>
+      </inertial>
+    </link>
+    <link name="left_foot">
+      <collision>
+        <origin xyz="0 0 0" rpy="0 0 0"/>
+        <geometry>
+          <mesh filename="package://legs_description/meshes/iteration_1/gazebo/left_foot_visual.stl"/>
+        </geometry>
+      </collision>
+      <visual>
+        <origin xyz="0 0 0" rpy="0 0 0"/>
+        <geometry>
+          <mesh filename="package://legs_description/meshes/iteration_1/gazebo/left_foot_visual.stl"/>
+        </geometry>
+        <material name="orange"/>
+      </visual>
+      <inertial>
+        <origin xyz="0 0 0" rpy="0 0 0"/>
+        <mass value="0.01"/>
+        <inertia
+          ixx="0.01" ixy="0.0" ixz="0.0"
+          iyy="0.01" iyz="0.0"
+          izz="0.01"/>
+      </inertial>
+    </link>
+    <link name="right_upper_limb">
+      <collision>
+        <origin xyz="0 0 0" rpy="0 0 0"/>
+        <geometry>
+          <mesh filename="package://legs_description/meshes/iteration_1/gazebo/right_upper_limb_visual.stl"/>
+        </geometry>
+      </collision>
+      <visual>
+        <origin xyz="0 0 0" rpy="0 0 0"/>
+        <geometry>
+          <mesh filename="package://legs_description/meshes/iteration_1/gazebo/right_upper_limb_visual.stl"/>
+        </geometry>
+        <material name="orange"/>
+      </visual>
+      <inertial>
+        <origin xyz="0 0 0" rpy="0 0 0"/>
+        <mass value="0.01"/>
+        <inertia
+          ixx="0.01" ixy="0.0" ixz="0.0"
+          iyy="0.01" iyz="0.0"
+          izz="0.01"/>
+      </inertial>
+    </link>
+    <link name="right_lower_limb">
+      <collision>
+        <origin xyz="0 0 0" rpy="0 0 0"/>
+        <geometry>
+          <mesh filename="package://legs_description/meshes/iteration_1/gazebo/right_lower_limb_visual.stl"/>
+        </geometry>
+      </collision>
+      <visual>
+        <origin xyz="0 0 0" rpy="0 0 0"/>
+        <geometry>
+          <mesh filename="package://legs_description/meshes/iteration_1/gazebo/right_lower_limb_visual.stl"/>
+        </geometry>
+        <material name="orange"/>
+      </visual>
+      <inertial>
+        <origin xyz="0 0 0" rpy="0 0 0"/>
+        <mass value="0.01"/>
+        <inertia
+          ixx="0.01" ixy="0.0" ixz="0.0"
+          iyy="0.01" iyz="0.0"
+          izz="0.01"/>
+      </inertial>
+    </link>
+    <link name="right_foot">
+      <collision>
+        <origin xyz="0 0 0" rpy="0 0 0"/>
+        <geometry>
+          <mesh filename="package://legs_description/meshes/iteration_1/gazebo/right_foot_visual.stl"/>
+        </geometry>
+      </collision>
+      <visual>
+        <origin xyz="0 0 0" rpy="0 0 0"/>
+        <geometry>
+          <mesh filename="package://legs_description/meshes/iteration_1/gazebo/right_foot_visual.stl"/>
+        </geometry>
+        <material name="orange"/>
+      </visual>
+      <inertial>
+        <origin xyz="0 0 0" rpy="0 0 0"/>
+        <mass value="0.01"/>
+        <inertia
+          ixx="0.01" ixy="0.0" ixz="0.0"
+          iyy="0.01" iyz="0.0"
+          izz="0.01"/>
+      </inertial>
+    </link>
   <!--
     Virtual links
   -->
   <link name="world"/>
-  <link name="plane_x">
+<!--   <link name="plane_x">
     <inertial>
       <mass value="2e-06"/>
       <inertia ixx="1.1e-09" ixy="0" ixz="0" iyy="1.1e-09" iyz="0" izz="1.1e-09"/>
     </inertial>
-  </link>
+  </link> -->
 	<!--
 		Joints
 	-->
-  <joint name="world_plane_x" type="planar">
+<!--   <joint name="world_plane_x" type="planar">
     <parent link="world"/>
     <child link="plane_x"/>
-    <origin xyz="0 0 ${footHeight + lowerLegHeight + upperLegHeight}" rpy="0 0 0"/>
+    <origin xyz="0 0 1" rpy="0 0 0"/>
     <axis xyz="1 0 0"/>
   </joint>
   <joint name="plane_x_body" type="continuous">
     <parent link="plane_x"/>
-    <child link="body"/>
+    <child link="hip"/>
     <origin xyz="0 0 0" rpy="0 0 0"/>
     <axis xyz="1 0 0"/>
-  </joint>
-	<joint name="left_hip" type="revolute">
-		<parent link="body"/>
-		<child link="left_upper_leg"/>
-		<origin xyz="${-legDistFromCenter} 0 0" rpy="0 ${PI/2} 0"/>
-		<axis xyz="0 0 1"/>
-		<limit effort="${upperLegLimitEffort}" velocity="${upperLegLimitVelocity}" lower="${upperLegLimitLowerPosition*DEG_TO_RAD}" upper="${upperLegLimitUpperPosition*DEG_TO_RAD}" />
-		<dynamics damping="${upperLegDamping}"/>
-	</joint>
-	<joint name="left_knee" type="revolute">
-		<parent link="left_upper_leg"/>
-		<child link="left_lower_leg"/>
-		<origin xyz="${upperLegHeight} 0 0" rpy="0 0 0"/>
-		<axis xyz="0 0 1"/>
-		<limit effort="${lowerLegLimitEffort}" velocity="${lowerLegLimitVelocity}" lower="${lowerLegLimitLowerPosition*DEG_TO_RAD}" upper="${lowerLegLimitUpperPosition*DEG_TO_RAD}" />
-		<dynamics damping="${lowerLegDamping}"/>
-	</joint>
-	<joint name="left_ankle" type="revolute">
-		<parent link="left_lower_leg"/>
-		<child link="left_foot"/>
-		<origin xyz="${lowerLegHeight} 0 0" rpy="0 0 0"/>
-		<axis xyz="0 0 1"/>
-		<limit effort="${footLimitEffort}" velocity="${footLimitVelocity}" lower="${footLimitLowerPosition*DEG_TO_RAD}" upper="${footLimitUpperPosition*DEG_TO_RAD}" />
-		<dynamics damping="${footDamping}"/>
-	</joint>
-	<joint name="right_hip" type="revolute">
-		<parent link="body"/>
-		<child link="right_upper_leg"/>
-		<origin xyz="${legDistFromCenter} 0 0" rpy="0 ${PI/2} 0"/>
-		<axis xyz="0 0 1"/>
+  </joint>  -->
+  <joint name="world_hip" type="fixed">
+    <parent link="world"/>
+    <child link="hip"/>
+    <origin xyz="0 0 1" rpy="0 0 0"/>
+  </joint>
+  <joint name="left_hip" type="revolute">
+    <parent link="hip"/>
+    <child link="left_upper_limb"/>
+    <origin xyz="0 0.0635 -0.028867" rpy="${-90*DEG_TO_RAD} 0 0"/>
+    <axis xyz="0 0 -1"/>
     <limit effort="${upperLegLimitEffort}" velocity="${upperLegLimitVelocity}" lower="${upperLegLimitLowerPosition*DEG_TO_RAD}" upper="${upperLegLimitUpperPosition*DEG_TO_RAD}" />
     <dynamics damping="${upperLegDamping}"/>
-	</joint>
-	<joint name="right_knee" type="revolute">
-		<parent link="right_upper_leg"/>
-		<child link="right_lower_leg"/>
-		<origin xyz="${upperLegHeight} 0 0" rpy="0 0 0"/>
-		<axis xyz="0 0 1"/>
+  </joint>
+  <joint name="left_knee" type="revolute">
+    <parent link="left_upper_limb"/>
+    <child link="left_lower_limb"/>
+    <origin xyz="0 0.262 0" rpy="0 0 0"/>
+    <axis xyz="0 0 -1"/>
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