Commit message: added scale for visual, mass and inertias components

File: src/legs_description/urdf/legs.xacro (robot description, xacro)
@@ -9,4 +9,7 @@
   <!-- Robot configuration: Miscellaneous -->
   <xacro:property name="robot_floating" value="0"/>
+  <xacro:property name="scale" value="10"/>
+  <xacro:property name="mass_scale" value="${pow(scale,3)}"/>
+  <xacro:property name="intertia_scale" value="${pow(scale,1.667)}"/>
 	<!-- Robot configuration: Transmission -->
 	<xacro:property name="max_real_motor_torque" value="1.0787315"/> <!-- In N*m -->
@@ -39,34 +42,34 @@
         <origin xyz="0 0 0" rpy="${90*DEG_TO_RAD} 0 0"/>
         <geometry>
-          <cylinder length="0.180" radius="0.025"/>
-        </geometry>
-      </collision>
-      <visual>
-        <origin xyz="0 0 0" rpy="0 0 0"/>
-        <geometry>
-          <mesh filename="package://legs_description/meshes/iteration_1/gazebo/hip_visual.stl"/>
-        </geometry>
-        <material name="orange"/>
-      </visual>
-      <inertial>
-        <origin xyz="0 0 0" rpy="0 0 0"/>
-        <mass value="0.156"/>
-        <inertia
-          ixx="3.03e-004" ixy="0.0" ixz="1.44e-008"
-          iyy="2.78e-005" iyz="0.0"
-          izz="3.14e-004"/>
+          <cylinder length="${scale*0.180}" radius="${scale*0.025}"/>
+        </geometry>
+      </collision>
+      <visual>
+        <origin xyz="0 0 0" rpy="0 0 0"/>
+        <geometry>
+          <mesh filename="package://legs_description/meshes/iteration_1/gazebo/hip_visual.stl" scale="${scale} ${scale} ${scale}"/>
+        </geometry>
+        <material name="orange"/>
+      </visual>
+      <inertial>
+        <origin xyz="0 0 0" rpy="0 0 0"/>
+        <mass value="${mass_scale*0.156}"/>
+        <inertia
+          ixx="${intertia_scale*3.03e-004}" ixy="${intertia_scale*0.0}" ixz="${intertia_scale*1.44e-008}"
+          iyy="${intertia_scale*2.78e-005}" iyz="${intertia_scale*0.0}"
+          izz="${intertia_scale*3.14e-004}"/>
       </inertial>
     </link>
     <link name="left_upper_limb">
       <collision>
-        <origin xyz="0 0.131 0" rpy="${90*DEG_TO_RAD} 0 0"/>
-        <geometry>
-          <cylinder length="0.262" radius="0.01"/>
-        </geometry>
-      </collision>
-      <visual>
-        <origin xyz="0 0 0" rpy="0 0 0"/>
-        <geometry>
-          <mesh filename="package://legs_description/meshes/iteration_1/gazebo/left_upper_limb_visual.stl"/>
+        <origin xyz="0 ${scale*0.131} 0" rpy="${90*DEG_TO_RAD} 0 0"/>
+        <geometry>
+          <cylinder length="${scale*0.262}" radius="${scale*0.01}"/>
+        </geometry>
+      </collision>
+      <visual>
+        <origin xyz="0 0 0" rpy="0 0 0"/>
+        <geometry>
+          <mesh filename="package://legs_description/meshes/iteration_1/gazebo/left_upper_limb_visual.stl" scale="${scale} ${scale} ${scale}"/>
         </geometry>
         <material name="orange"/>
@@ -74,32 +77,32 @@
       <inertial>
         <origin xyz="0 0 0" rpy="90 0 0"/>
-        <mass value="0.123"/>
-        <inertia
-          ixx="1.19e-003" ixy="2.89e-006" ixz="-1.36e-008"
-          iyy="1.69e-005" iyz="-1.78e-005"
-          izz="1.18e-003"/>
+        <mass value="${mass_scale*0.123}"/>
+        <inertia
+          ixx="${intertia_scale*1.19e-003}" ixy="${intertia_scale*2.89e-006}" ixz="${intertia_scale*-1.36e-008}"
+          iyy="${intertia_scale*1.69e-005}" iyz="${intertia_scale*-1.78e-005}"
+          izz="${intertia_scale*1.18e-003}"/>
       </inertial>
     </link>
     <link name="left_lower_limb">
       <collision>
-        <origin xyz="0 0.131 0" rpy="${90*DEG_TO_RAD} 0 0"/>
-        <geometry>
-          <cylinder length="0.212" radius="0.01"/>
-        </geometry>
-      </collision>
-      <visual>
-        <origin xyz="0 0 0" rpy="0 0 0"/>
-        <geometry>
-          <mesh filename="package://legs_description/meshes/iteration_1/gazebo/left_lower_limb_visual.stl"/>
-        </geometry>
-        <material name="orange"/>
-      </visual>
-      <inertial>
-        <origin xyz="0 0 0" rpy="0 0 0"/>
-        <mass value="0.115"/>
-        <inertia
-          ixx="6.99e-004" ixy="2.44e-005" ixz="0.0"
-          iyy="1.85e-005" iyz="-1.82e-005"
-          izz="6.94e-004"/>
+        <origin xyz="0 ${scale*0.106} 0" rpy="${90*DEG_TO_RAD} 0 0"/>
+        <geometry>
+          <cylinder length="${scale*0.212}" radius="${scale*0.01}"/>
+        </geometry>
+      </collision>
+      <visual>
+        <origin xyz="0 0 0" rpy="0 0 0"/>
+        <geometry>
+          <mesh filename="package://legs_description/meshes/iteration_1/gazebo/left_lower_limb_visual.stl" scale="${scale} ${scale} ${scale}"/>
+        </geometry>
+        <material name="orange"/>
+      </visual>
+      <inertial>
+        <origin xyz="0 0 0" rpy="0 0 0"/>
+        <mass value="${mass_scale*0.115}"/>
+        <inertia
+          ixx="${intertia_scale*6.99e-004}" ixy="${intertia_scale*2.44e-005}" ixz="${intertia_scale*0.0}"
+          iyy="${intertia_scale*1.85e-005}" iyz="${intertia_scale*-1.82e-005}"
+          izz="${intertia_scale*6.94e-004}"/>
       </inertial>
     </link>
@@ -108,67 +111,67 @@
         <origin xyz="0 0 0" rpy="0 0 0"/>
         <geometry>
-          <mesh filename="package://legs_description/meshes/iteration_1/gazebo/left_foot_visual.stl"/>
-        </geometry>
-      </collision>
-      <visual>
-        <origin xyz="0 0 0" rpy="0 0 0"/>
-        <geometry>
-          <mesh filename="package://legs_description/meshes/iteration_1/gazebo/left_foot_visual.stl"/>
-        </geometry>
-        <material name="orange"/>
-      </visual>
-      <inertial>
-        <origin xyz="0 0 0" rpy="0 0 0"/>
-        <mass value="0.021"/>
-        <inertia
-          ixx="2.2e-005" ixy="-9.16e-006" ixz="0.0"
-          iyy="-9.16e-006" iyz="9.05e-006"
-          izz="2.88e-005"/>
+          <mesh filename="package://legs_description/meshes/iteration_1/gazebo/left_foot_visual.stl" scale="${scale} ${scale} ${scale}"/>
+        </geometry>
+      </collision>
+      <visual>
+        <origin xyz="0 0 0" rpy="0 0 0"/>
+        <geometry>
+          <mesh filename="package://legs_description/meshes/iteration_1/gazebo/left_foot_visual.stl" scale="${scale} ${scale} ${scale}"/>
+        </geometry>
+        <material name="orange"/>
+      </visual>
+      <inertial>
+        <origin xyz="0 0 0" rpy="0 0 0"/>
+        <mass value="${mass_scale*0.021}"/>
+        <inertia
+          ixx="${intertia_scale*2.2e-005}" ixy="${intertia_scale*-9.16e-006}" ixz="${intertia_scale*0.0}"
+          iyy="${intertia_scale*-9.16e-006}" iyz="${intertia_scale*9.05e-006}"
+          izz="${intertia_scale*2.88e-005}"/>
       </inertial>
     </link>
     <link name="right_upper_limb">
       <collision>
-        <origin xyz="0 0.131 0" rpy="${90*DEG_TO_RAD} 0 0"/>
-        <geometry>
-          <cylinder length="0.262" radius="0.01"/>
-        </geometry>
-      </collision>
-      <visual>
-        <origin xyz="0 0 0" rpy="0 0 0"/>
-        <geometry>
-          <mesh filename="package://legs_description/meshes/iteration_1/gazebo/right_upper_limb_visual.stl"/>
-        </geometry>
-        <material name="orange"/>
-      </visual>
-      <inertial>
-        <origin xyz="0 0 0" rpy="0 0 0"/>
-        <mass value="0.123"/>
-        <inertia
-          ixx="1.19e-003" ixy="2.89e-006" ixz="-1.36e-008"
-          iyy="1.69e-005" iyz="-1.78e-005"
-          izz="1.18e-003"/>
+        <origin xyz="0 ${scale*0.131} 0" rpy="${90*DEG_TO_RAD} 0 0"/>
+        <geometry>
+          <cylinder length="${scale*0.262}" radius="${scale*0.01}"/>
+        </geometry>
+      </collision>
+      <visual>
+        <origin xyz="0 0 0" rpy="0 0 0"/>
+        <geometry>
+          <mesh filename="package://legs_description/meshes/iteration_1/gazebo/right_upper_limb_visual.stl" scale="${scale} ${scale} ${scale}"/>
+        </geometry>
+        <material name="orange"/>
+      </visual>
+      <inertial>
+        <origin xyz="0 0 0" rpy="0 0 0"/>
+        <mass value="${mass_scale*0.123}"/>
+        <inertia
+          ixx="${intertia_scale*1.19e-003}" ixy="${intertia_scale*2.89e-006}" ixz="${intertia_scale*-1.36e-008}"
+          iyy="${intertia_scale*1.69e-005}" iyz="${intertia_scale*-1.78e-005}"
+          izz="${intertia_scale*1.18e-003}"/>
       </inertial>
     </link>
     <link name="right_lower_limb">
       <collision>
-        <origin xyz="0 0.131 0" rpy="${90*DEG_TO_RAD} 0 0"/>
-        <geometry>
-          <cylinder length="0.212" radius="0.01"/>
-        </geometry>
-      </collision>
-      <visual>
-        <origin xyz="0 0 0" rpy="0 0 0"/>
-        <geometry>
-          <mesh filename="package://legs_description/meshes/iteration_1/gazebo/right_lower_limb_visual.stl"/>
-        </geometry>
-        <material name="orange"/>
-      </visual>
-      <inertial>
-        <origin xyz="0 0 0" rpy="0 0 0"/>
-        <mass value="0.115"/>
-        <inertia
-          ixx="6.99e-004" ixy="2.44e-005" ixz="0.0"
-          iyy="1.85e-005" iyz="-1.82e-005"
-          izz="6.94e-004"/>
+        <origin xyz="0 ${scale*0.106} 0" rpy="${90*DEG_TO_RAD} 0 0"/>
+        <geometry>
+          <cylinder length="${scale*0.212}" radius="${scale*0.01}"/>
+        </geometry>
+      </collision>
+      <visual>
+        <origin xyz="0 0 0" rpy="0 0 0"/>
+        <geometry>
+          <mesh filename="package://legs_description/meshes/iteration_1/gazebo/right_lower_limb_visual.stl" scale="${scale} ${scale} ${scale}"/>
+        </geometry>
+        <material name="orange"/>
+      </visual>
+      <inertial>
+        <origin xyz="0 0 0" rpy="0 0 0"/>
+        <mass value="${mass_scale*0.115}"/>
+        <inertia
+          ixx="${intertia_scale*6.99e-004}" ixy="${intertia_scale*2.44e-005}" ixz="${intertia_scale*0.0}"
+          iyy="${intertia_scale*1.85e-005}" iyz="${intertia_scale*-1.82e-005}"
+          izz="${intertia_scale*6.94e-004}"/>
       </inertial>
     </link>
@@ -177,21 +180,21 @@
         <origin xyz="0 0 0" rpy="0 0 0"/>
         <geometry>
-          <mesh filename="package://legs_description/meshes/iteration_1/gazebo/right_foot_visual.stl"/>
-        </geometry>
-      </collision>
-      <visual>
-        <origin xyz="0 0 0" rpy="0 0 0"/>
-        <geometry>
-          <mesh filename="package://legs_description/meshes/iteration_1/gazebo/right_foot_visual.stl"/>
-        </geometry>
-        <material name="orange"/>
-      </visual>
-      <inertial>
-        <origin xyz="0 0 0" rpy="0 0 0"/>
-        <mass value="0.021"/>
-        <inertia
-          ixx="2.2e-005" ixy="-9.16e-006" ixz="0.0"
-          iyy="-9.16e-006" iyz="9.05e-006"
-          izz="2.88e-005"/>
+          <mesh filename="package://legs_description/meshes/iteration_1/gazebo/right_foot_visual.stl" scale="${scale} ${scale} ${scale}"/>
+        </geometry>
+      </collision>
+      <visual>
+        <origin xyz="0 0 0" rpy="0 0 0"/>
+        <geometry>
+          <mesh filename="package://legs_description/meshes/iteration_1/gazebo/right_foot_visual.stl" scale="${scale} ${scale} ${scale}"/>
+        </geometry>
+        <material name="orange"/>
+      </visual>
+      <inertial>
+        <origin xyz="0 0 0" rpy="0 0 0"/>
+        <mass value="${mass_scale*0.021}"/>
+        <inertia
+          ixx="${intertia_scale*2.2e-005}" ixy="${intertia_scale*-9.16e-006}" ixz="${intertia_scale*0.0}"
+          iyy="${intertia_scale*-9.16e-006}" iyz="${intertia_scale*9.05e-006}"
+          izz="${intertia_scale*2.88e-005}"/>
       </inertial>
     </link>
@@ -202,6 +205,6 @@
 <!--   <link name="world_pris">
     <inertial>
-      <mass value="2e-06"/>
-      <inertia ixx="1.1e-09" ixy="0" ixz="0" iyy="1.1e-09" iyz="0" izz="1.1e-09"/>
+      <mass value="${mass_scale*2e-06"/>
+      <inertia ixx="${intertia_scale*1.1e-09" ixy="${intertia_scale*0" ixz="${intertia_scale*0" iyy="${intertia_scale*1.1e-09" iyz="${intertia_scale*0" izz="${intertia_scale*1.1e-09"/>
     </inertial>
   </link>
@@ -218,11 +221,11 @@
     <child link="hip"/>
     <axis xyz="0 1 0"/>
-  </joint> -->
-<!--
+  </joint>
   <joint name="world_hip" type="continuous">
     <origin xyz="0 0 1" rpy="0 0 0"/>
     <parent link="world"/>
     <child link="hip"/>
-  </joint>  -->
+  </joint>
+  -->
 	<!--
 		Joints
@@ -231,5 +234,5 @@
     <parent link="hip"/>
     <child link="left_upper_limb"/>
-    <origin xyz="0 0.0635 -0.028867" rpy="${-90*DEG_TO_RAD} 0 0"/>
+    <origin xyz="0 ${scale*0.0635} ${scale*-0.028867}" rpy="${-90*DEG_TO_RAD} 0 0"/>
     <axis xyz="0 0 -1"/>
     <limit effort="${upperLegLimitEffort}" velocity="${upperLegLimitVelocity}" lower="${upperLegLimitLowerPosition*DEG_TO_RAD}" upper="${upperLegLimitUpperPosition*DEG_TO_RAD}" />
@@ -239,5 +242,5 @@
     <parent link="left_upper_limb"/>
     <child link="left_lower_limb"/>
-    <origin xyz="0 0.262 0" rpy="0 0 0"/>
+    <origin xyz="0 ${scale*0.262} 0" rpy="0 0 0"/>
     <axis xyz="0 0 -1"/>
     <limit effort="${lowerLegLimitEffort}" velocity="${lowerLegLimitVelocity}" lower="${lowerLegLimitLowerPosition*DEG_TO_RAD}" upper="${lowerLegLimitUpperPosition*DEG_TO_RAD}" />
@@ -247,5 +250,5 @@
     <parent link="left_lower_limb"/>
     <child link="left_foot"/>
-    <origin xyz="0 0.212 0" rpy="0 0 0"/>
+    <origin xyz="0 ${scale*0.212} 0" rpy="0 0 0"/>
     <axis xyz="0 0 -1"/>
     <limit effort="${footLimitEffort}" velocity="${footLimitVelocity}" lower="${footLimitLowerPosition*DEG_TO_RAD}" upper="${footLimitUpperPosition*DEG_TO_RAD}" />
@@ -255,5 +258,5 @@
     <parent link="hip"/>
     <child link="right_upper_limb"/>
-    <origin xyz="0 -0.0635 -0.028867" rpy="${-90*DEG_TO_RAD} 0 0"/>
+    <origin xyz="0 ${scale*-0.0635} ${scale*-0.028867}" rpy="${-90*DEG_TO_RAD} 0 0"/>
     <axis xyz="0 0 -1"/>
     <limit effort="${upperLegLimitEffort}" velocity="${upperLegLimitVelocity}" lower="${upperLegLimitLowerPosition*DEG_TO_RAD}" upper="${upperLegLimitUpperPosition*DEG_TO_RAD}" />
@@ -263,5 +266,5 @@
     <parent link="right_upper_limb"/>
     <child link="right_lower_limb"/>
-    <origin xyz="0 0.262 0" rpy="0 0 0"/>
+    <origin xyz="0 ${scale*0.262} 0" rpy="0 0 0"/>
     <axis xyz="0 0 -1"/>
     <limit effort="${lowerLegLimitEffort}" velocity="${lowerLegLimitVelocity}" lower="${lowerLegLimitLowerPosition*DEG_TO_RAD}" upper="${lowerLegLimitUpperPosition*DEG_TO_RAD}" />
@@ -271,5 +274,5 @@
     <parent link="right_lower_limb"/>
     <child link="right_foot"/>
-    <origin xyz="0 0.212 0" rpy="0 0 0"/>
+    <origin xyz="0 ${scale*0.212} 0" rpy="0 0 0"/>
     <axis xyz="0 0 -1"/>
     <limit effort="${footLimitEffort}" velocity="${footLimitVelocity}" lower="${footLimitLowerPosition*DEG_TO_RAD}" upper="${footLimitUpperPosition*DEG_TO_RAD}" />
@@ -341,9 +344,8 @@
     <xacro:property name="rotational_robot_holder_base_length_extra" value="0.1" />
   </xacro:if>
-  <xacro:property name="rotational_robot_holder_base_length" value="1" />
-  <xacro:property name="rotational_robot_holder_base_radius" value="0.2" />
-  <xacro:property name="rotational_robot_holder_holder_radius" value="0.01" />
-  <xacro:property name="rotational_robot_holder_holder_length" value="2" />
-  <!-- <xacro:include filename="$(find gazebo_resources)/models/rotational_robot_holder/urdf/rotational_robot_holder.xacro" /> -->
+  <xacro:property name="rotational_robot_holder_base_length" value="${scale*0.67}" />
+  <xacro:property name="rotational_robot_holder_base_radius" value="${scale*0.2}" />
+  <xacro:property name="rotational_robot_holder_holder_radius" value="${scale*0.01}" />
+  <xacro:property name="rotational_robot_holder_holder_length" value="${scale*2}" />
   <link name="rotational_robot_holder_base">
     <collision>
@@ -362,5 +364,5 @@
     <inertial>
       <mass value="10"/>
-      <inertia ixx="0.4" ixy="0.0" ixz="0.0" iyy="0.4" iyz="0.0" izz="0.2"/>
+      <inertia ixx="0.002" ixy="0.0" ixz="0.0" iyy="0.002" iyz="0.0" izz="0.002"/>
     </inertial>
   </link>
@@ -381,5 +383,5 @@
     <inertial>
       <mass value="0.01"/>
-      <inertia ixx="0.1" ixy="0.0" ixz="0.0" iyy="0.1" iyz="0.0" izz="0.1"/>
+      <inertia ixx="0.002" ixy="0.0" ixz="0.0" iyy="0.002" iyz="0.0" izz="0.002"/>
     </inertial>
   </link>
@@ -400,8 +402,7 @@
     <inertial>
       <mass value="0.01"/>
-      <inertia ixx="0.1" ixy="0.0" ixz="0.0" iyy="0.1" iyz="0.0" izz="0.1"/>
+      <inertia ixx="0.002" ixy="0.0" ixz="0.0" iyy="0.002" iyz="0.0" izz="0.002"/>
     </inertial>
   </link>
-  <!-- Robot to rotational_robot_holder -->
   <joint name="rotational_robot_holder_base_to_world" type="fixed">
     <parent link="world"/>
