Commit message: fixed some bugs and added flag for using the rotational holder or just have the robot floating

File: src/legs_description/urdf/legs.xacro (robot description, xacro)
@@ -9,4 +9,5 @@
   <!-- Robot configuration: Miscellaneous -->
   <xacro:property name="robot_floating" value="0"/>
+  <xacro:property name="rotational_holder" value="0"/>
   <xacro:property name="scale" value="1"/>
   <xacro:property name="mass_scale" value="${pow(scale,3)}"/>
@@ -76,5 +77,5 @@
       </visual>
       <inertial>
-        <origin xyz="0 0 0" rpy="90 0 0"/>
+        <origin xyz="0 0 0" rpy="0 0 0"/>
         <mass value="${mass_scale*0.123}"/>
         <inertia
@@ -125,8 +126,8 @@
         <mass value="${mass_scale*0.021}"/>
         <inertia
-          ixx="0.0" ixy="0.0" ixz="0.0"
-          iyy="0.0" iyz="0.0"
-          izz="0.0"/>
-      </inertial>
+          ixx="${intertia_scale*2.2e-005}" ixy="0.0" ixz="0.0"
+          iyy="0.0" iyz="0.0"
+          izz="${intertia_scale*2.88e-005}"/>
+        </inertial>
     </link>
     <link name="right_upper_limb">
@@ -197,5 +198,5 @@
           iyy="0.0" iyz="0.0"
           izz="${intertia_scale*2.88e-005}"/>
-      </inertial>
+        </inertial>
     </link>
   <!--
@@ -203,29 +204,30 @@
   -->
   <link name="world"/>
-<!--   <link name="world_pris">
-    <inertial>
-      <mass value="${mass_scale*2e-06"/>
-      <inertia ixx="${intertia_scale*1.1e-09" ixy="${intertia_scale*0" ixz="${intertia_scale*0" iyy="${intertia_scale*1.1e-09" iyz="${intertia_scale*0" izz="${intertia_scale*1.1e-09"/>
-    </inertial>
-  </link>
-  <joint name="world_world_pris" type="prismatic">
-    <origin xyz="0 0 1" rpy="0 0 0"/>
-    <parent link="world"/>
-    <child link="world_pris"/>
-    <axis xyz="0 0 1"/>
-    <limit effort="1000" velocity="1000" lower="0" upper="5" />
-  </joint>
-  <joint name="world_pris_hip" type="continuous">
-    <origin xyz="0 0 0" rpy="0 0 0"/>
-    <parent link="world_pris"/>
-    <child link="hip"/>
-    <axis xyz="0 1 0"/>
-  </joint>
-  <joint name="world_hip" type="continuous">
-    <origin xyz="0 0 1" rpy="0 0 0"/>
-    <parent link="world"/>
-    <child link="hip"/>
-  </joint>
-  -->
+  <xacro:if value="${rotational_holder is 0}">
+<!--     <link name="world_pris">
+      <inertial>
+        <mass value="2e-06"/>
+        <inertia ixx="0.002" ixy="0" ixz="0" iyy="0.002" iyz="0" izz="0.002"/>
+      </inertial>
+    </link>
+    <joint name="world_world_pris" type="prismatic">
+      <origin xyz="0 0 1" rpy="0 0 0"/>
+      <parent link="world"/>
+      <child link="world_pris"/>
+      <axis xyz="0 0 1"/>
+      <limit effort="1000" velocity="1000" lower="0" upper="5" />
+    </joint>
+    <joint name="world_pris_hip" type="continuous">
+      <origin xyz="0 0 0" rpy="0 0 0"/>
+      <parent link="world_pris"/>
+      <child link="hip"/>
+      <axis xyz="0 1 0"/>
+    </joint>  -->
+    <joint name="world_hip" type="floating">
+      <origin xyz="0 0 0.54" rpy="0 0 0"/>
+      <parent link="world"/>
+      <child link="hip"/>
+    </joint>
+  </xacro:if>
 	<!--
 		Joints
@@ -250,5 +252,5 @@
     <parent link="left_lower_limb"/>
     <child link="left_foot"/>
-    <origin xyz="0 ${scale*0.212} 0" rpy="0 0 0"/>
+    <origin xyz="0 ${scale*0.212} 0" rpy="0 0 ${-90*DEG_TO_RAD}"/>
     <axis xyz="0 0 -1"/>
     <limit effort="${footLimitEffort}" velocity="${footLimitVelocity}" lower="${footLimitLowerPosition*DEG_TO_RAD}" upper="${footLimitUpperPosition*DEG_TO_RAD}" />
@@ -274,5 +276,5 @@
     <parent link="right_lower_limb"/>
     <child link="right_foot"/>
-    <origin xyz="0 ${scale*0.212} 0" rpy="0 0 0"/>
+    <origin xyz="0 ${scale*0.212} 0" rpy="0 0 ${-90*DEG_TO_RAD}"/>
     <axis xyz="0 0 -1"/>
     <limit effort="${footLimitEffort}" velocity="${footLimitVelocity}" lower="${footLimitLowerPosition*DEG_TO_RAD}" upper="${footLimitUpperPosition*DEG_TO_RAD}" />
@@ -340,105 +342,107 @@
   </transmission>
   <!-- Rotational robot holder -->
-  <xacro:property name="rotational_robot_holder_base_length_extra" value="0" />
-  <xacro:if value="${robot_floating is 1}">
-    <xacro:property name="rotational_robot_holder_base_length_extra" value="0.1" />
+  <xacro:if value="${rotational_holder is 1}">
+    <xacro:property name="rotational_robot_holder_base_length_extra" value="0" />
+    <xacro:if value="${robot_floating is 1}">
+      <xacro:property name="rotational_robot_holder_base_length_extra" value="0.1" />
+    </xacro:if>
+    <xacro:property name="rotational_robot_holder_base_length" value="${scale*0.67}" />
+    <xacro:property name="rotational_robot_holder_base_radius" value="${scale*0.2}" />
+    <xacro:property name="rotational_robot_holder_holder_radius" value="${scale*0.01}" />
+    <xacro:property name="rotational_robot_holder_holder_length" value="${scale*2}" />
+    <link name="rotational_robot_holder_base">
+      <collision>
+        <origin xyz="0 0 0" rpy="0 0 0"/>
+        <geometry>
+          <cylinder length="${rotational_robot_holder_base_length}" radius="${rotational_robot_holder_base_radius}"/>
+        </geometry>
+      </collision>
+      <visual>
+        <origin xyz="0 0 0" rpy="0 0 0"/>
+        <geometry>
+          <cylinder length="${rotational_robot_holder_base_length}" radius="${rotational_robot_holder_base_radius}"/>
+        </geometry>
+        <material name="orange"/>
+      </visual>
+      <inertial>
+        <mass value="10"/>
+        <inertia ixx="0.002" ixy="0.0" ixz="0.0" iyy="0.002" iyz="0.0" izz="0.002"/>
+      </inertial>
+    </link>
+    <link name="rotational_robot_holder_virtual">
+      <collision>
+        <origin xyz="0 0 0" rpy="0 0 0"/>
+        <geometry>
+          <sphere radius="0.01"/>
+        </geometry>
+      </collision>
+      <visual>
+        <origin xyz="0 0 0" rpy="0 0 0"/>
+        <geometry>
+           <sphere radius="0.01"/>
+        </geometry>
+        <material name="orange"/>
+      </visual>
+      <inertial>
+        <mass value="0.001"/>
+        <inertia ixx="0.002" ixy="0.0" ixz="0.0" iyy="0.002" iyz="0.0" izz="0.002"/>
+      </inertial>
+    </link>
+    <link name="rotational_robot_holder_holder">
+      <collision>
+        <origin xyz="${rotational_robot_holder_holder_length/2} 0 0" rpy="0 ${PI/2} 0"/>
+        <geometry>
+          <cylinder length="${rotational_robot_holder_holder_length}" radius="${rotational_robot_holder_holder_radius}"/>
+        </geometry>
+      </collision>
+      <visual>
+        <origin xyz="${rotational_robot_holder_holder_length/2} 0 0" rpy="0 ${PI/2} 0"/>
+        <geometry>
+           <cylinder length="${rotational_robot_holder_holder_length}" radius="${rotational_robot_holder_holder_radius}"/>
+        </geometry>
+        <material name="orange"/>
+      </visual>
+      <inertial>
+        <mass value="0.001"/>
+        <inertia ixx="0.002" ixy="0.0" ixz="0.0" iyy="0.002" iyz="0.0" izz="0.002"/>
+      </inertial>
+    </link>
+    <joint name="rotational_robot_holder_base_to_world" type="fixed">
+      <parent link="world"/>
+      <child link="rotational_robot_holder_base"/>
+      <origin xyz="0 0 ${rotational_robot_holder_base_length/2}" rpy="0 0 0"/>
+    </joint>
+    <xacro:if value="${robot_floating is 1}">
+      <joint name="rotational_robot_holder_virtual_to_holder" type="fixed">
+        <parent link="rotational_robot_holder_base"/>
+        <child link="rotational_robot_holder_virtual"/>
+      </joint>
+      <joint name="rotational_robot_holder_joint" type="fixed">
+        <parent link="rotational_robot_holder_virtual"/>
+        <child link="rotational_robot_holder_holder"/>
+        <origin xyz="0 0 ${rotational_robot_holder_base_length/2}" rpy="0 0 0"/>
+      </joint>
+    </xacro:if>
+    <xacro:if value="${robot_floating is 0}">
+      <joint name="rotational_robot_holder_virtual_to_holder" type="continuous">
+        <parent link="rotational_robot_holder_base"/>
+        <child link="rotational_robot_holder_virtual"/>
+        <origin xyz="0 0 0" rpy="0 0 0"/>
+        <axis xyz="0 1 0"/>
+      </joint>
+      <joint name="rotational_robot_holder_joint" type="continuous">
+        <parent link="rotational_robot_holder_virtual"/>
+        <child link="rotational_robot_holder_holder"/>
+        <origin xyz="0 0 ${rotational_robot_holder_base_length/2}" rpy="0 0 0"/>
+        <axis xyz="0 0 1"/>
+      </joint>
+    </xacro:if>
+    <joint name="rotational_robot_holder_to_rotot" type="fixed">
+      <parent link="rotational_robot_holder_holder"/>
+      <child link="hip"/>
+      <origin xyz="${rotational_robot_holder_holder_length+0.2} 0 0" rpy="0 0 ${90*DEG_TO_RAD}"/>
+      <axis xyz="0 0 1"/>
+      <limit effort="30" velocity="2.0" lower="0" upper="1" />
+    </joint>
   </xacro:if>
-  <xacro:property name="rotational_robot_holder_base_length" value="${scale*0.67}" />
-  <xacro:property name="rotational_robot_holder_base_radius" value="${scale*0.2}" />
-  <xacro:property name="rotational_robot_holder_holder_radius" value="${scale*0.01}" />
-  <xacro:property name="rotational_robot_holder_holder_length" value="${scale*2}" />
-  <link name="rotational_robot_holder_base">
-    <collision>
-      <origin xyz="0 0 0" rpy="0 0 0"/>
-      <geometry>
-        <cylinder length="${rotational_robot_holder_base_length}" radius="${rotational_robot_holder_base_radius}"/>
-      </geometry>
-    </collision>
-    <visual>
-      <origin xyz="0 0 0" rpy="0 0 0"/>
-      <geometry>
-        <cylinder length="${rotational_robot_holder_base_length}" radius="${rotational_robot_holder_base_radius}"/>
-      </geometry>
-      <material name="orange"/>
-    </visual>
-    <inertial>
-      <mass value="10"/>
-      <inertia ixx="0.002" ixy="0.0" ixz="0.0" iyy="0.002" iyz="0.0" izz="0.002"/>
-    </inertial>
-  </link>
-  <link name="rotational_robot_holder_virtual">
-    <collision>
-      <origin xyz="0 0 0" rpy="0 0 0"/>
-      <geometry>
-        <sphere radius="0.01"/>
-      </geometry>
-    </collision>
-    <visual>
-      <origin xyz="0 0 0" rpy="0 0 0"/>
-      <geometry>
-         <sphere radius="0.01"/>
-      </geometry>
-      <material name="orange"/>
-    </visual>
-    <inertial>
-      <mass value="0.001"/>
-      <inertia ixx="0.002" ixy="0.0" ixz="0.0" iyy="0.002" iyz="0.0" izz="0.002"/>
-    </inertial>
-  </link>
-  <link name="rotational_robot_holder_holder">
-    <collision>
-      <origin xyz="${rotational_robot_holder_holder_length/2} 0 0" rpy="0 ${PI/2} 0"/>
-      <geometry>
-        <cylinder length="${rotational_robot_holder_holder_length}" radius="${rotational_robot_holder_holder_radius}"/>
-      </geometry>
-    </collision>
-    <visual>
-      <origin xyz="${rotational_robot_holder_holder_length/2} 0 0" rpy="0 ${PI/2} 0"/>
-      <geometry>
-         <cylinder length="${rotational_robot_holder_holder_length}" radius="${rotational_robot_holder_holder_radius}"/>
-      </geometry>
-      <material name="orange"/>
-    </visual>
-    <inertial>
-      <mass value="0.001"/>
-      <inertia ixx="0.002" ixy="0.0" ixz="0.0" iyy="0.002" iyz="0.0" izz="0.002"/>
-    </inertial>
-  </link>
-  <joint name="rotational_robot_holder_base_to_world" type="fixed">
-    <parent link="world"/>
-    <child link="rotational_robot_holder_base"/>
-    <origin xyz="0 0 ${rotational_robot_holder_base_length/2}" rpy="0 0 0"/>
-  </joint>
-  <xacro:if value="${robot_floating is 1}">
-    <joint name="rotational_robot_holder_virtual_to_holder" type="fixed">
-      <parent link="rotational_robot_holder_base"/>
-      <child link="rotational_robot_holder_virtual"/>
-    </joint>
-    <joint name="rotational_robot_holder_joint" type="fixed">
-      <parent link="rotational_robot_holder_virtual"/>
-      <child link="rotational_robot_holder_holder"/>
-      <origin xyz="0 0 ${rotational_robot_holder_base_length/2}" rpy="0 0 0"/>
-    </joint>
-  </xacro:if>
-  <xacro:if value="${robot_floating is 0}">
-    <joint name="rotational_robot_holder_virtual_to_holder" type="continuous">
-      <parent link="rotational_robot_holder_base"/>
-      <child link="rotational_robot_holder_virtual"/>
-      <origin xyz="0 0 0" rpy="0 0 0"/>
-      <axis xyz="0 1 0"/>
-    </joint>
-    <joint name="rotational_robot_holder_joint" type="continuous">
-      <parent link="rotational_robot_holder_virtual"/>
-      <child link="rotational_robot_holder_holder"/>
-      <origin xyz="0 0 ${rotational_robot_holder_base_length/2}" rpy="0 0 0"/>
-      <axis xyz="0 0 1"/>
-    </joint>
-  </xacro:if>
-  <joint name="rotational_robot_holder_to_rotot" type="fixed">
-    <parent link="rotational_robot_holder_holder"/>
-    <child link="hip"/>
-    <origin xyz="${rotational_robot_holder_holder_length+0.2} 0 0" rpy="0 0 ${90*DEG_TO_RAD}"/>
-    <axis xyz="0 0 1"/>
-    <limit effort="30" velocity="2.0" lower="0" upper="1" />
-  </joint>
 </robot>

Commit message: fixed joint limits of the ankle

File: src/legs_description/urdf/legs.xacro (robot description, xacro)
@@ -29,6 +29,6 @@
   <xacro:property name="lowerLegLimitVelocity" value="10" />
   <xacro:property name="lowerLegLimitEffort" value="10" />
-  <xacro:property name="footLimitUpperPosition" value="120" />
-  <xacro:property name="footLimitLowerPosition" value="-50" />
+  <xacro:property name="footLimitUpperPosition" value="30" />
+  <xacro:property name="footLimitLowerPosition" value="-80" />
   <xacro:property name="footLimitVelocity" value="10" />
   <xacro:property name="footLimitEffort" value="10" />

Commit message: improved rotational holder

File: src/legs_description/urdf/legs.xacro (robot description, xacro)
@@ -9,5 +9,5 @@
   <!-- Robot configuration: Miscellaneous -->
   <xacro:property name="robot_floating" value="0"/>
-  <xacro:property name="rotational_holder" value="0"/>
+  <xacro:property name="rotational_holder" value="1"/>
   <xacro:property name="scale" value="1"/>
   <xacro:property name="mass_scale" value="${pow(scale,3)}"/>
@@ -347,7 +347,7 @@
       <xacro:property name="rotational_robot_holder_base_length_extra" value="0.1" />
     </xacro:if>
-    <xacro:property name="rotational_robot_holder_base_length" value="${scale*0.67}" />
-    <xacro:property name="rotational_robot_holder_base_radius" value="${scale*0.2}" />
-    <xacro:property name="rotational_robot_holder_holder_radius" value="${scale*0.01}" />
+    <xacro:property name="rotational_robot_holder_base_length" value="${scale*0.54}" />
+    <xacro:property name="rotational_robot_holder_base_radius" value="${scale*0.1}" />
+    <xacro:property name="rotational_robot_holder_holder_radius" value="${scale*0.005}" />
     <xacro:property name="rotational_robot_holder_holder_length" value="${scale*2}" />
     <link name="rotational_robot_holder_base">
@@ -366,6 +366,9 @@
       </visual>
       <inertial>
-        <mass value="10"/>
-        <inertia ixx="0.002" ixy="0.0" ixz="0.0" iyy="0.002" iyz="0.0" izz="0.002"/>
+        <mass value="0.001"/>
+        <inertia
+          ixx="2e-005" ixy="0.0" ixz="0.0"
+          iyy="0.0" iyz="0.0"
+          izz="2e-005"/>
       </inertial>
     </link>
@@ -386,6 +389,9 @@
       <inertial>
         <mass value="0.001"/>
-        <inertia ixx="0.002" ixy="0.0" ixz="0.0" iyy="0.002" iyz="0.0" izz="0.002"/>
-      </inertial>
+        <inertia
+          ixx="2e-005" ixy="0.0" ixz="0.0"
+          iyy="0.0" iyz="0.0"
+          izz="2e-005"/>
+        </inertial>
     </link>
     <link name="rotational_robot_holder_holder">
@@ -405,6 +411,9 @@
       <inertial>
         <mass value="0.001"/>
-        <inertia ixx="0.002" ixy="0.0" ixz="0.0" iyy="0.002" iyz="0.0" izz="0.002"/>
-      </inertial>
+        <inertia
+          ixx="2e-005" ixy="0.0" ixz="0.0"
+          iyy="0.0" iyz="0.0"
+          izz="2e-005"/>
+        </inertial>
     </link>
     <joint name="rotational_robot_holder_base_to_world" type="fixed">
@@ -441,5 +450,5 @@
       <parent link="rotational_robot_holder_holder"/>
       <child link="hip"/>
-      <origin xyz="${rotational_robot_holder_holder_length+0.2} 0 0" rpy="0 0 ${90*DEG_TO_RAD}"/>
+      <origin xyz="${rotational_robot_holder_holder_length+0.1} 0 0" rpy="0 0 ${90*DEG_TO_RAD}"/>
       <axis xyz="0 0 1"/>
       <limit effort="30" velocity="2.0" lower="0" upper="1" />

Commit message: fixed scaling factors

File: src/legs_description/urdf/legs.xacro (robot description, xacro)
@@ -9,8 +9,8 @@
   <!-- Robot configuration: Miscellaneous -->
   <xacro:property name="robot_floating" value="0"/>
-  <xacro:property name="rotational_holder" value="1"/>
+  <xacro:property name="rotational_holder" value="0"/>
   <xacro:property name="scale" value="1"/>
   <xacro:property name="mass_scale" value="${pow(scale,3)}"/>
-  <xacro:property name="intertia_scale" value="${pow(scale,1.667)}"/>
+  <xacro:property name="intertia_scale" value="${pow(scale,5)}"/>
 	<!-- Robot configuration: Transmission -->
 	<xacro:property name="max_real_motor_torque" value="1.0787315"/> <!-- In N*m -->

Commit message: using rotational holder

File: src/legs_description/urdf/legs.xacro (robot description, xacro)
@@ -9,5 +9,5 @@
   <!-- Robot configuration: Miscellaneous -->
   <xacro:property name="robot_floating" value="0"/>
-  <xacro:property name="rotational_holder" value="0"/>
+  <xacro:property name="rotational_holder" value="1"/>
   <xacro:property name="scale" value="1"/>
   <xacro:property name="mass_scale" value="${pow(scale,3)}"/>
